File: KiCAD/L-STAT.sch (KiCad schematic (older format))
At the start: 73 parts

Commit message: System did some house keeping on exit.
Signed-off-by: John Bradley <flypie@rocketmail.com>
Parts:
- RV-L-STAT-36: renamed from R-L-STAT-?; footprint (none) -> Potentiometer_THT:3362H1103LF
- V-L-STAT-3, V-L-STAT-7, V-L-STAT-8: value CV173 -> VR91
- gave numbers to parts that had none: 53
- renumbered V-L-STAT-2 to V-L-STAT-1
