File: KiCAD/KEYSW1.sch (KiCad schematic (older format))
At the start: 21 parts

Commit message: kvpsu2.pdf
Parts:
- removed Fn-KEYSW1-? (x2), L-KEYSW1-? (x3): SW_SPDT, SamacSys_Parts_m:A101SYCQ04, symbol Switch:SW_SPDT
- removed J-KEYSW1-?: CL.4, SamacSys_Parts_l:242431, symbol Connector:Conn_01x01_Female
- removed SW-KEYSW1-?: SW_DPDT_x2, SamacSys_Parts_m:7205SYCQE, symbol Switch:SW_DPDT_x2
- added Fn-KEYSW1-1, Fn-KEYSW1-3, L-KEYSW1-1, L-KEYSW1-2, L-KEYSW1-3: SW_SPDT, SamacSys_Parts_m:A101SYCQ04, symbol Switch:SW_SPDT
- added J-KEYSW1-3: CL.4, SamacSys_Parts_l:242431, symbol Connector:Conn_01x01_Female
- added unit 2 of SW-KEYSW1-2
- gave numbers to parts that had none: 14
Connections:
- net AUTO\MAN.CMN2: now also SW-KEYSW1-2.5 (B)
- net AUTO\MAN.NC2: now also SW-KEYSW1-2.4 (A)
- net at Fn-KEYSW1-2.3 (C), L-KEYSW1-4.3 (C), L-KEYSW1-5.3 (C)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: now also Fn-KEYSW1-1.3 (C), Fn-KEYSW1-3.3 (C), L-KEYSW1-1.3 (C), L-KEYSW1-2.3 (C), L-KEYSW1-3.3 (C)
- net at J-KEYSW1-4.1 (Pin_1): now also L-KEYSW1-2.2 (B)
- net at J-KEYSW1-5.1 (Pin_1): now also L-KEYSW1-3.2 (B)
- net at J-KEYSW1-8.1 (Pin_1): now also Fn-KEYSW1-1.2 (B)
- net at J-KEYSW1-10.1 (Pin_1): now also Fn-KEYSW1-3.2 (B)
- new net: J-KEYSW1-3.1 (Pin_1), L-KEYSW1-1.2 (B)
Changed lines of the file:
@@
 $Descr A4 11693 8268
 encoding utf-8
-Sheet 22 24
+Sheet 22 25
 Title "Key Switches 1 Position 4.6"
-Date ""
+Date "2020-10-08"
 Rev "Alpha"
 Comp "John Bradley"
@@
 $EndDescr
 $Comp
-L Switch:SW_SPDT L-KEYSW1-?
-U 1 1 5F6DEACB
+L Switch:SW_SPDT L-KEYSW1-1
+U 1 1 5F8BCA5D
 P 3900 2800
-F 0 "L-KEYSW1-?" H 3900 3100 50  0000 C CNN
+F 0 "L-KEYSW1-1" H 3900 3100 50  0000 C CNN
 F 1 "SW_SPDT" H 3900 3000 50  0000 C CNN
 F 2 "SamacSys_Parts_m:A101SYCQ04" H 3900 2800 50  0001 C CNN
@@
 	4100 2800 4100 1250
 $Comp
-L Switch:SW_SPDT L-KEYSW1-?
-U 1 1 5F6DF0AF
+L Switch:SW_SPDT L-KEYSW1-2
+U 1 1 5F8BCA5E
 P 4550 2800
-F 0 "L-KEYSW1-?" H 4550 3100 50  0000 C CNN
+F 0 "L-KEYSW1-2" H 4550 3100 50  0000 C CNN
 F 1 "SW_SPDT" H 4550 3000 50  0000 C CNN
 F 2 "SamacSys_Parts_m:A101SYCQ04" H 4550 2800 50  0001 C CNN
@@
 $EndComp
 $Comp
-L Switch:SW_SPDT L-KEYSW1-?
-U 1 1 5F6DF68F
+L Switch:SW_SPDT L-KEYSW1-3
+U 1 1 5F8BCA5F
 P 5200 2800
-F 0 "L-KEYSW1-?" H 5200 3100 50  0000 C CNN
+F 0 "L-KEYSW1-3" H 5200 3100 50  0000 C CNN
 F 1 "SW_SPDT" H 5200 3000 50  0000 C CNN
 F 2 "SamacSys_Parts_m:A101SYCQ04" H 5200 2800 50  0001 C CNN
@@
 $EndComp
 $Comp
-L Switch:SW_SPDT L-KEYSW1-?
+L Switch:SW_SPDT L-KEYSW1-4
 U 1 1 5F6DF69A
 P 5850 2800
-F 0 "L-KEYSW1-?" H 5850 3100 50  0000 C CNN
+F 0 "L-KEYSW1-4" H 5850 3100 50  0000 C CNN
 F 1 "SW_SPDT" H 5850 3000 50  0000 C CNN
 F 2 "SamacSys_Parts_m:A101SYCQ04" H 5850 2800 50  0001 C CNN
@@
 	6050 2800 6050 2000
 $Comp
-L Switch:SW_SPDT L-KEYSW1-?
+L Switch:SW_SPDT L-KEYSW1-5
 U 1 1 5F6E060B
 P 6500 2800
-F 0 "L-KEYSW1-?" H 6500 3100 50  0000 C CNN
+F 0 "L-KEYSW1-5" H 6500 3100 50  0000 C CNN
 F 1 "SW_SPDT" H 6500 3000 50  0000 C CNN
 F 2 "SamacSys_Parts_m:A101SYCQ04" H 6500 2800 50  0001 C CNN
@@
 	4100 1250 7050 1250
 $Comp
-L Connector:Conn_01x01_Female J-KEYSW1-?
-U 1 1 5F6E867D
+L Connector:Conn_01x01_Female J-KEYSW1-3
+U 1 1 5F8BCA62
 P 7250 1250
-F 0 "J-KEYSW1-?" H 7300 1300 50  0000 L CNN
+F 0 "J-KEYSW1-3" H 7300 1300 50  0000 L CNN
 F 1 "CL.4" H 7300 1200 50  0000 L CNN
 F 2 "SamacSys_Parts_l:242431" H 7250 1250 50  0001 C CNN
@@
 $EndComp
 $Comp
-L Connector:Conn_01x01_Female J-KEYSW1-?
+L Connector:Conn_01x01_Female J-KEYSW1-4
 U 1 1 5F6E9647
 P 7250 1500
-F 0 "J-KEYSW1-?" H 7300 1550 50  0000 L CNN
+F 0 "J-KEYSW1-4" H 7300 1550 50  0000 L CNN
 F 1 "CL.3" H 7300 1450 50  0000 L CNN
 F 2 "SamacSys_Parts_l:242431" H 7250 1500 50  0001 C CNN
@@
 $EndComp
 $Comp
-L Connector:Conn_01x01_Female J-KEYSW1-?
+L Connector:Conn_01x01_Female J-KEYSW1-5
 U 1 1 5F6E9885
 P 7250 1750
-F 0 "J-KEYSW1-?" H 7300 1800 50  0000 L CNN
+F 0 "J-KEYSW1-5" H 7300 1800 50  0000 L CNN
 F 1 "CL.2" H 7300 1700 50  0000 L CNN
 F 2 "SamacSys_Parts_l:242431" H 7250 1750 50  0001 C CNN
@@
 $EndComp
 $Comp
-L Connector:Conn_01x01_Female J-KEYSW1-?
+L Connector:Conn_01x01_Female J-KEYSW1-6
 U 1 1 5F6E9B0F
 P 7250 2000
-F 0 "J-KEYSW1-?" H 7300 2050 50  0000 L CNN
+F 0 "J-KEYSW1-6" H 7300 2050 50  0000 L CNN
 F 1 "CL.1" H 7300 1950 50  0000 L CNN
 F 2 "SamacSys_Parts_l:242431" H 7250 2000 50  0001 C CNN
@@
 $EndComp
 $Comp
-L Connector:Conn_01x01_Female J-KEYSW1-?
+L Connector:Conn_01x01_Female J-KEYSW1-7
 U 1 1 5F6E9D68
 P 7250 2250
-F 0 "J-KEYSW1-?" H 7300 2300 50  0000 L CNN
+F 0 "J-KEYSW1-7" H 7300 2300 50  0000 L CNN
 F 1 "CL.0" H 7300 2200 50  0000 L CNN
 F 2 "SamacSys_Parts_l:242431" H 7250 2250 50  0001 C CNN
@@
 $EndComp
 $Comp
-L Switch:SW_SPDT Fn-KEYSW1-?
-U 1 1 5F6EF1E2
+L Switch:SW_SPDT Fn-KEYSW1-1
+U 1 1 5F8BCA67
 P 3900 3800
-F 0 "Fn-KEYSW1-?" H 3900 4100 50  0000 C CNN
+F 0 "Fn-KEYSW1-1" H 3900 4100 50  0000 C CNN
 F 1 "SW_SPDT" H 3900 4000 50  0000 C CNN
 F 2 "SamacSys_Parts_m:A101SYCQ04" H 3900 3800 50  0001 C CNN
@@
 $EndComp
 $Comp
-L Switch:SW_SPDT Fn-KEYSW1-?
+L Switch:SW_SPDT Fn-KEYSW1-2
 U 1 1 5F6EFB91
 P 4550 3800
-F 0 "Fn-KEYSW1-?" H 4550 4100 50  0000 C CNN
+F 0 "Fn-KEYSW1-2" H 4550 4100 50  0000 C CNN
 F 1 "SW_SPDT" H 4550 4000 50  0000 C CNN
 F 2 "SamacSys_Parts_m:A101SYCQ04" H 4550 3800 50  0001 C CNN
@@
 $EndComp
 $Comp
-L Switch:SW_SPDT Fn-KEYSW1-?
-U 1 1 5F6EFFA9
+L Switch:SW_SPDT Fn-KEYSW1-3
+U 1 1 5F8BCA69
 P 5200 3800
-F 0 "Fn-KEYSW1-?" H 5200 4100 50  0000 C CNN
+F 0 "Fn-KEYSW1-3" H 5200 4100 50  0000 C CNN
 F 1 "SW_SPDT" H 5200 4000 50  0000 C CNN
 F 2 "SamacSys_Parts_m:A101SYCQ04" H 5200 3800 50  0001 C CNN
@@
 	3700 4100 4350 4100
 $Comp
-L Connector:Conn_01x01_Female J-KEYSW1-?
+L Connector:Conn_01x01_Female J-KEYSW1-8
 U 1 1 5F6F23CD
 P 7250 3200
-F 0 "J-KEYSW1-?" H 7300 3250 50  0000 L CNN
+F 0 "J-KEYSW1-8" H 7300 3250 50  0000 L CNN
 F 1 "CL.15" H 7300 3150 50  0000 L CNN
 F 2 "SamacSys_Parts_l:242431" H 7250 3200 50  0001 C CNN
@@
 $EndComp
 $Comp
-L Connector:Conn_01x01_Female J-KEYSW1-?
+L Connector:Conn_01x01_Female J-KEYSW1-9
 U 1 1 5F6F23D7
 P 7250 3450
-F 0 "J-KEYSW1-?" H 7300 3500 50  0000 L CNN
+F 0 "J-KEYSW1-9" H 7300 3500 50  0000 L CNN
 F 1 "CL.14" H 7300 3400 50  0000 L CNN
 F 2 "SamacSys_Parts_l:242431" H 7250 3450 50  0001 C CNN
@@
 $EndComp
 $Comp
-L Connector:Conn_01x01_Female J-KEYSW1-?
+L Connector:Conn_01x01_Female J-KEYSW1-10
 U 1 1 5F6F23E1
 P 7250 3700
-F 0 "J-KEYSW1-?" H 7300 3750 50  0000 L CNN
+F 0 "J-KEYSW1-10" H 7300 3750 50  0000 L CNN
 F 1 "CL.13" H 7300 3650 50  0000 L CNN
 F 2 "SamacSys_Parts_l:242431" H 7250 3700 50  0001 C CNN
@@
 	5400 3400 6900 3400
 $Comp
-L Switch:SW_DPDT_x2 SW-KEYSW1-?
+L Switch:SW_DPDT_x2 SW-KEYSW1-2
 U 1 1 5F6FA300
 P 3900 4800
-F 0 "SW-KEYSW1-?" H 3900 5100 50  0000 C CNN
+F 0 "SW-KEYSW1-2" H 3900 5100 50  0000 C CNN
 F 1 "SW_DPDT_x2" H 3900 5000 50  0000 C CNN
 F 2 "SamacSys_Parts_m:7205SYCQE" H 3900 4800 50  0001 C CNN
@@
 $EndComp
 $Comp
-L Switch:SW_DPDT_x2 SW-KEYSW1-?
-U 2 1 5F6FAB6D
+L Switch:SW_DPDT_x2 SW-KEYSW1-2
+U 2 1 5F8BCA6E
 P 5250 4800
-F 0 "SW-KEYSW1-?" H 5250 5100 50  0000 C CNN
+F 0 "SW-KEYSW1-2" H 5250 5100 50  0000 C CNN
 F 1 "SW_DPDT_x2" H 5250 5000 50  0000 C CNN
 F 2 "SamacSys_Parts_m:7205SYCQE" H 5250 4800 50  0001 C CNN
@@
 NoConn ~ 5000 3700
 $Comp
-L Switch:SW_Push SW-KEYSW1-?
+L Switch:SW_Push SW-KEYSW1-1
 U 1 1 5F6D7B97
 P 2350 1500
-F 0 "SW-KEYSW1-?" H 2350 1800 50  0000 C CNN
+F 0 "SW-KEYSW1-1" H 2350 1800 50  0000 C CNN
 F 1 "SW_Push" H 2350 1700 50  0000 C CNN
 F 2 "Button_Switch_THT:SW_PUSH-12mm" H 2350 1700 50  0001 C CNN
@@
 	2150 1500 1900 1500
 $Comp
-L Connector:Conn_01x01_Female J-KEYSW1-?
+L Connector:Conn_01x01_Female J-KEYSW1-2
 U 1 1 5F6D9736
 P 2950 1500
-F 0 "J-KEYSW1-?" H 3000 1550 50  0000 L CNN
+F 0 "J-KEYSW1-2" H 3000 1550 50  0000 L CNN
 F 1 "Hs" H 3000 1450 50  0000 L CNN
 F 2 "SamacSys_Parts_l:242431" H 2950 1500 50  0001 C CNN
@@
 $EndComp
 $Comp
-L Connector:Conn_01x01_Female J-KEYSW1-?
+L Connector:Conn_01x01_Female J-KEYSW1-1
 U 1 1 5F6D9DF1
 P 1700 1500
-F 0 "J-KEYSW1-?" H 1750 1550 50  0000 L CNN
+F 0 "J-KEYSW1-1" H 1750 1550 50  0000 L CNN
 F 1 "SUP.ACT.LN" H 1750 1450 50  0000 L CNN
 F 2 "SamacSys_Parts_l:242431" H 1700 1500 50  0001 C CNN
