File: KiCAD/KEYSW2.sch (KiCad schematic (older format))
At the start: 33 parts

Commit message: kvpsu2.pdf
Parts:
- removed Fn-KEYSW2-?, L-KEYSW2-? (x2): SW_SPDT, SamacSys_Parts_m:A101SYCQ04, symbol Switch:SW_SPDT
- removed J-KEYSW2-?: CL.3, SamacSys_Parts_l:242431, symbol Connector:Conn_01x01_Female
- removed J-KEYSW2-?: CL.2, SamacSys_Parts_l:242431, symbol Connector:Conn_01x01_Female
- removed J-KEYSW2-?: CL.1, SamacSys_Parts_l:242431, symbol Connector:Conn_01x01_Female
- removed J-KEYSW2-?: CL.0, SamacSys_Parts_l:242431, symbol Connector:Conn_01x01_Female
- removed J-KEYSW2-?: CL.15, SamacSys_Parts_l:242431, symbol Connector:Conn_01x01_Female
- removed J-KEYSW2-?: CL.14, SamacSys_Parts_l:242431, symbol Connector:Conn_01x01_Female
- removed J-KEYSW2-?: CL.13, SamacSys_Parts_l:242431, symbol Connector:Conn_01x01_Female
- removed SW-KEYSW2-?: SW_DPDT_x2, SamacSys_Parts_m:7205SYCQE, symbol Switch:SW_DPDT_x2
- added Fn-KEYSW2-2, L-KEYSW2-4, L-KEYSW2-5: SW_SPDT, SamacSys_Parts_m:A101SYCQ04, symbol Switch:SW_SPDT
- added J-KEYSW2-2: CL.3, SamacSys_Parts_l:242431, symbol Connector:Conn_01x01_Female
- added J-KEYSW2-3: CL.2, SamacSys_Parts_l:242431, symbol Connector:Conn_01x01_Female
- added J-KEYSW2-4: CL.1, SamacSys_Parts_l:242431, symbol Connector:Conn_01x01_Female
- added J-KEYSW2-5: CL.0, SamacSys_Parts_l:242431, symbol Connector:Conn_01x01_Female
- added J-KEYSW2-6: CL.15, SamacSys_Parts_l:242431, symbol Connector:Conn_01x01_Female
- added J-KEYSW2-7: CL.14, SamacSys_Parts_l:242431, symbol Connector:Conn_01x01_Female
- added J-KEYSW2-8: CL.13, SamacSys_Parts_l:242431, symbol Connector:Conn_01x01_Female
- added unit 1 of SW-KEYSW2-1
- L-KEYSW2-16: renamed from SW?; footprint (none) -> Connector_PinHeader_2.54mm:PinHeader_1x04_P2.54mm_Vertical
- R-KEYSW2-1: footprint (none) -> Resistor_THT:R_Axial_DIN0516_L15.5mm_D5.0mm_P5.08mm_Vertical
- R-KEYSW2-2: renamed from R-KEYSW2-?; footprint (none) -> Resistor_THT:R_Axial_DIN0516_L15.5mm_D5.0mm_P5.08mm_Vertical
- gave numbers to parts that had none: 19

Commit message: Finish KEYSW2/ Add extra Symbols for switches.
Signed-off-by: John Bradley <flypie@rocketmail.com>
Parts:
- removed Fn-KEYSW2-1, Fn-KEYSW2-2, Fn-KEYSW2-3, L-KEYSW2-1, L-KEYSW2-10, L-KEYSW2-11, L-KEYSW2-12, L-KEYSW2-13, L-KEYSW2-14, L-KEYSW2-15, L-KEYSW2-2, L-KEYSW2-3, L-KEYSW2-4, L-KEYSW2-5, L-KEYSW2-8, L-KEYSW2-9: SW_SPDT, SamacSys_Parts_m:A101SYCQ04, symbol Switch:SW_SPDT
- removed J-KEYSW2-7: CL.14, SamacSys_Parts_l:242431, symbol Connector:Conn_01x01_Female
- removed J-KEYSW2-8: CL.13, SamacSys_Parts_l:242431, symbol Connector:Conn_01x01_Female
- removed L-KEYSW2-16: SW_Push_Dual, Connector_PinHeader_2.54mm:PinHeader_1x04_P2.54mm_Vertical, symbol Switch:SW_Push_Dual
- removed S2: 7205SYCQE, 7205SYCQE, symbol SamacSys_Parts:7205SYCQE
- removed SW-KEYSW2-1: SW_DPDT_x2, SamacSys_Parts_m:7205SYCQE, symbol Switch:SW_DPDT_x2
- added SW-KEYSW2-1, SW-KEYSW2-2: SW_QPDT, Connector_PinHeader_2.54mm:PinHeader_1x12_P2.54mm_Vertical, symbol NEWValves:SW_QPDT
- added SW-KEYSW2-16: SW_Double_Acting_Push, Connector_PinHeader_2.54mm:PinHeader_1x04_P2.54mm_Vertical, symbol NEWValves:SW_Double_Acting_Push
- added SW-KEYSW2-4, SW-KEYSW2-5: SW_Push_DPDT, Connector_PinHeader_2.54mm:PinHeader_1x06_P2.54mm_Vertical, symbol Switch:SW_Push_DPDT
- added SW10, SW6, SW7, SW8, SW9: SW_Push, Connector_PinHeader_2.54mm:PinHeader_1x02_P2.54mm_Vertical, symbol Switch:SW_Push
- J-KEYSW2-1: value CL.4 -> KM.cmn
- J-KEYSW2-2: value CL.3 -> B
- J-KEYSW2-3: value CL.2 -> M
- J-KEYSW2-4: value CL.1 -> MON.S
- J-KEYSW2-5: value CL.0 -> MON.A
- J-KEYSW2-6: value CL.15 -> MON.C
- R-KEYSW2-2: value 47K -> 100K
- SW-KEYSW2-3: renamed from S1; symbol SamacSys_Parts:7205SYCQE -> Switch:SW_Push_DPDT
Connections:
- net labels added: A.ERASE, AC.ERASE, C.ERASE, CSINHIBIT, HS, KC.CMN, KC.NC, KC.NO, KLC, Minus.30v, PC.Read, S.ERASE, S.ERASE.ALL, S.ERASE.LINE, STOP.RUN, Stop.Noise
- net labels removed: AUTO\MAN.CMN2, AUTO\MAN.NC2, CI&CR.CF, HA.CF
- wire segments 58 -> 71
- no-connect marks 11 -> 27
Other:
- note added: "CS"
- note added: "Completion Signal\nChassis"
- note added: "Erase"
- note added: "From Stop\nChassis"
- note added: "KAC"
- note added: "KCC"
- note added: "KMC"
- note added: "KSC"
- note added: "Monitor Switches"
- note added: "RUN"
- note added: "STOP"
- note added: "To Acc\nStore Gate"
- note added: "To C.S.\nChassis"
- note added: "To Control\nStore Gate"
- note added: "To Inward\nTransfer Gate"
- note added: "To Monitor Chassis"
- note added: "To PC Interface"
- note added: "To PC\nInterface"
- note added: "To Write/Erase\nChassis"
- note added: "Write"
- note added: "Write/\nErase"
- moved on the sheet: L-KEYSW2-6, L-KEYSW2-7
