File: KiCAD/SSEMD.kicad_pcb (KiCad board)
At the start: 2 copper layers, 1112 parts, among them U1 L78L05_TO92

Commit message: kvpsu2.pdf
Parts:
- removed Fn-KEYSW1-0, L-KEYSW1-0: SW_SPDT, SamacSys_Parts_m:A101SYCQ04
- added C-KVPSU1-1: 1.5uf 3kV, Capacitor_THT:C_Disc_D7.5mm_W5.0mm_P5.00mm, F.Cu at (608.4, 102.8)
- added C-KVPSU1-2: 1.5uf 3kV, Capacitor_THT:C_Disc_D7.5mm_W5.0mm_P5.00mm, F.Cu at (618.7, 94.8)
- added C-KVPSU1-3: 0.5, Capacitor_THT:C_Disc_D7.5mm_W5.0mm_P5.00mm, F.Cu at (588.0, 125.9)
- added C-KVPSU1-4: 0.5, Capacitor_THT:C_Disc_D7.5mm_W5.0mm_P5.00mm, F.Cu at (577.7, 138.0)
- added C-KVPSU1-5: 0.5uf 3kv, Capacitor_THT:C_Disc_D7.5mm_W5.0mm_P5.00mm, F.Cu at (600.1, 119.3)
- added C-KVPSU1-6: 0.5uf 3kv, Capacitor_THT:C_Disc_D7.5mm_W5.0mm_P5.00mm, F.Cu at (608.4, 109.3)
- added C-KVPSU1-7: 0.5, Capacitor_THT:C_Disc_D7.5mm_W5.0mm_P5.00mm, F.Cu at (587.7, 132.4)
- added C-KVPSU1-8: 0.5, Capacitor_THT:C_Disc_D7.5mm_W5.0mm_P5.00mm, F.Cu at (618.7, 101.3)
- added C-KVPSU1-9: 0.5uf 3kv, Capacitor_THT:C_Disc_D7.5mm_W5.0mm_P5.00mm, F.Cu at (627.8, 93.8)
- added C-KVPSU2-1: 1.5uf 3kV, Capacitor_THT:C_Disc_D7.5mm_W5.0mm_P5.00mm, F.Cu at (609.5, 407.9)
- added C-KVPSU2-2: 4.5uf 1.5kV, Capacitor_THT:C_Disc_D7.5mm_W5.0mm_P5.00mm, F.Cu at (618.6, 410.7)
- added C-KVPSU2-3: 4.5uf 1.5kV, Capacitor_THT:C_Disc_D7.5mm_W5.0mm_P5.00mm, F.Cu at (650.4, 378.7)
- added F-KVPSU1-1: 4A, Fuse:Fuse_Littelfuse_395Series, F.Cu at (623.7, 87.7)
- added F-KVPSU1-2: 4A, Fuse:Fuse_Littelfuse_395Series, F.Cu at (578.1, 131.9)
- added F-KVPSU2-1: 4A, Fuse:Fuse_Littelfuse_395Series, F.Cu at (655.5, 365.0)
- added F-KVPSU2-2: 4A, Fuse:Fuse_Littelfuse_395Series, F.Cu at (655.5, 359.4)
- added Fn-KEYSW1-3: SW_SPDT, SamacSys_Parts_m:A101SYCQ04, F.Cu at (655.9, 325.0)
- added Fn-KEYSW2-1: SW_SPDT, SamacSys_Parts_m:A101SYCQ04, F.Cu at (533.2, 381.7)
- added Fn-KEYSW2-2: SW_SPDT, SamacSys_Parts_m:A101SYCQ04, F.Cu at (485.4, 376.1)
- added Fn-KEYSW2-3: SW_SPDT, SamacSys_Parts_m:A101SYCQ04, F.Cu at (512.5, 348.4)
- added J-KEYSW2-1: CL.4, SamacSys_Parts_l:242431, F.Cu at (444.8, 365.9)
- added J-KEYSW2-2: CL.3, SamacSys_Parts_l:242431, F.Cu at (471.9, 352.0)
- added J-KEYSW2-3: CL.2, SamacSys_Parts_l:242431, F.Cu at (499.0, 338.2)
- added J-KEYSW2-4: CL.1, SamacSys_Parts_l:242431, F.Cu at (444.8, 379.7)
- added J-KEYSW2-5: CL.0, SamacSys_Parts_l:242431, F.Cu at (471.9, 365.9)
- added J-KEYSW2-6: CL.15, SamacSys_Parts_l:242431, F.Cu at (471.9, 338.2)
- added J-KEYSW2-7: CL.14, SamacSys_Parts_l:242431, F.Cu at (444.8, 352.0)
- added J-KEYSW2-8: CL.13, SamacSys_Parts_l:242431, F.Cu at (444.8, 338.2)
- added J-KVPSU1-1: L, SamacSys_Parts_l:242431, F.Cu at (500.3, 129.4)
- added J-KVPSU1-10: S.EHT -KV, SamacSys_Parts_l:242431, F.Cu at (529.0, 128.2)
- added J-KVPSU1-2: N, SamacSys_Parts_l:242431, F.Cu at (589.6, 85.7)
- added J-KVPSU1-3: E, SamacSys_Parts_l:242431, F.Cu at (556.1, 114.5)
- added J-KVPSU1-4: +4V L, SamacSys_Parts_l:242431, F.Cu at (589.6, 71.9)
- added J-KVPSU1-5: +4V N, SamacSys_Parts_l:242431, F.Cu at (560.8, 99.6)
- added J-KVPSU1-6: +4V L, SamacSys_Parts_l:242431, F.Cu at (533.7, 100.7)
- added J-KVPSU1-7: +4V N, SamacSys_Parts_l:242431, F.Cu at (562.5, 85.7)
- added J-KVPSU1-8: JA77847, Connector_PinHeader_2.54mm:PinHeader_1x08_P2.54mm_Vertical, F.Cu at (552.7, 124.0)
- added J-KVPSU1-9: 0V, SamacSys_Parts_l:242431, F.Cu at (562.5, 71.9)
- added J-KVPSU2-1: L, SamacSys_Parts_l:242431, F.Cu at (627.1, 377.1)
- added J-KVPSU2-2: N, SamacSys_Parts_l:242431, F.Cu at (598.3, 390.9)
- added J-KVPSU2-3: E, SamacSys_Parts_l:242431, F.Cu at (627.1, 363.3)
- added J-KVPSU2-4: +4V L, SamacSys_Parts_l:242431, F.Cu at (571.2, 405.9)
- added J-KVPSU2-5: 0V, SamacSys_Parts_l:242431, F.Cu at (571.2, 392.0)
- added J-KVPSU2-6: M.EHT, SamacSys_Parts_l:242431, F.Cu at (600.0, 377.1)
- added J-KVPSU2-7: +4V N, SamacSys_Parts_l:242431, F.Cu at (600.0, 363.3)
- added L-KEYSW1-5: SW_SPDT, SamacSys_Parts_m:A101SYCQ04, F.Cu at (665.5, 325.0)
- added L-KEYSW2-1: SW_SPDT, SamacSys_Parts_m:A101SYCQ04, F.Cu at (550.7, 350.0)
- added L-KEYSW2-10: SW_SPDT, SamacSys_Parts_m:A101SYCQ04, F.Cu at (504.5, 380.2)
- added L-KEYSW2-11: SW_SPDT, SamacSys_Parts_m:A101SYCQ04, F.Cu at (517.1, 366.3)
- added L-KEYSW2-12: SW_SPDT, SamacSys_Parts_m:A101SYCQ04, F.Cu at (495.0, 380.2)
- added L-KEYSW2-13: SW_SPDT, SamacSys_Parts_m:A101SYCQ04, F.Cu at (539.6, 334.6)
- added L-KEYSW2-14: SW_SPDT, SamacSys_Parts_m:A101SYCQ04, F.Cu at (507.6, 364.8)
- added L-KEYSW2-15: SW_SPDT, SamacSys_Parts_m:A101SYCQ04, F.Cu at (522.1, 350.9)
- added L-KEYSW2-16: SW_Push_Dual, Connector_PinHeader_2.54mm:PinHeader_1x04_P2.54mm_Vertical, F.Cu at (543.3, 364.7)
- added L-KEYSW2-2: SW_SPDT, SamacSys_Parts_m:A101SYCQ04, F.Cu at (523.6, 381.7)
- added L-KEYSW2-3: SW_SPDT, SamacSys_Parts_m:A101SYCQ04, F.Cu at (536.2, 366.3)
- added L-KEYSW2-4: SW_SPDT, SamacSys_Parts_m:A101SYCQ04, F.Cu at (526.7, 366.3)
- added L-KEYSW2-5: SW_SPDT, SamacSys_Parts_m:A101SYCQ04, F.Cu at (541.2, 350.0)
- added L-KEYSW2-6: SW_SPDT, SamacSys_Parts_m:A101SYCQ04, F.Cu at (514.1, 381.7)
- added L-KEYSW2-7: SW_SPDT, SamacSys_Parts_m:A101SYCQ04, F.Cu at (531.6, 350.9)
- added L-KEYSW2-8: SW_SPDT, SamacSys_Parts_m:A101SYCQ04, F.Cu at (498.0, 364.8)
- added L-KEYSW2-9: SW_SPDT, SamacSys_Parts_m:A101SYCQ04, F.Cu at (549.2, 334.6)
- added L-KVPSU1-1: 100h 20 mA, Connector_PinHeader_2.54mm:PinHeader_1x02_P2.54mm_Vertical, F.Cu at (544.5, 137.7)
- added L-KVPSU2-1: 100h 20 mA, Connector_PinHeader_2.54mm:PinHeader_1x02_P2.54mm_Vertical, F.Cu at (646.2, 386.6)
- added M-KVPSU1-1: Voltmeter_DC, Connector_PinHeader_2.54mm:PinHeader_1x02_P2.54mm_Vertical, F.Cu at (517.4, 139.0)
- added MES-KVPSU2-1: 2.5 KV, Connector_PinHeader_2.54mm:PinHeader_1x02_P2.54mm_Vertical, F.Cu at (661.0, 370.1)
- added R-KEYSW2-1: 47K, Resistor_THT:R_Axial_DIN0516_L15.5mm_D5.0mm_P5.08mm_Vertical, F.Cu at (452.6, 390.2)
- added R-KEYSW2-2: 47K, Resistor_THT:R_Axial_DIN0516_L15.5mm_D5.0mm_P5.08mm_Vertical, F.Cu at (442.3, 390.2)
- added R-KVPSU1-1: 2R 3W, Resistor_THT:R_Axial_DIN0516_L15.5mm_D5.0mm_P5.08mm_Vertical, F.Cu at (508.1, 139.9)
- added R-KVPSU1-10: 22K, Resistor_THT:R_Axial_DIN0516_L15.5mm_D5.0mm_P5.08mm_Vertical, F.Cu at (614.1, 75.1)
- added R-KVPSU1-11: 470, Resistor_THT:R_Axial_DIN0516_L15.5mm_D5.0mm_P5.08mm_Vertical, F.Cu at (535.2, 138.7)
- added R-KVPSU1-12: 470, Resistor_THT:R_Axial_DIN0516_L15.5mm_D5.0mm_P5.08mm_Vertical, F.Cu at (497.7, 139.9)
- added R-KVPSU1-13: 470k, Resistor_THT:R_Axial_DIN0516_L15.5mm_D5.0mm_P5.08mm_Vertical, F.Cu at (558.3, 138.1)
- added R-KVPSU1-14: 470k, Resistor_THT:R_Axial_DIN0516_L15.5mm_D5.0mm_P5.08mm_Vertical, F.Cu at (568.6, 125.0)
- added R-KVPSU1-15: 47k 2W, Resistor_THT:R_Axial_DIN0516_L15.5mm_D5.0mm_P5.08mm_Vertical, F.Cu at (624.5, 68.6)
- added R-KVPSU1-16: 15k 3W, Resistor_THT:R_Axial_DIN0516_L15.5mm_D5.0mm_P5.08mm_Vertical, F.Cu at (580.7, 119.3)
- added R-KVPSU1-17: 2R 3W, Resistor_THT:R_Axial_DIN0516_L15.5mm_D5.0mm_P5.08mm_Vertical, F.Cu at (624.5, 75.1)
- added R-KVPSU1-18: 360k, Resistor_THT:R_Axial_DIN0516_L15.5mm_D5.0mm_P5.08mm_Vertical, F.Cu at (609.7, 96.2)
- added R-KVPSU1-19: 15k 3W, Resistor_THT:R_Axial_DIN0516_L15.5mm_D5.0mm_P5.08mm_Vertical, F.Cu at (624.5, 81.7)
- added R-KVPSU1-2: 0R8 4W, Resistor_THT:R_Axial_DIN0516_L15.5mm_D5.0mm_P5.08mm_Vertical, F.Cu at (568.6, 131.5)
- added R-KVPSU1-20: 4.5m, Resistor_THT:R_Axial_DIN0207_L6.3mm_D2.5mm_P2.54mm_Vertical, F.Cu at (597.0, 124.6)
- added R-KVPSU1-21: 15k 3W, Resistor_THT:R_Axial_DIN0516_L15.5mm_D5.0mm_P5.08mm_Vertical, F.Cu at (591.0, 119.3)
- added R-KVPSU1-22: 4.7k, Resistor_THT:R_Axial_DIN0516_L15.5mm_D5.0mm_P5.08mm_Vertical, F.Cu at (614.1, 81.7)
- added R-KVPSU1-3: 470K, Resistor_THT:R_Axial_DIN0516_L15.5mm_D5.0mm_P5.08mm_Vertical, F.Cu at (524.8, 138.7)
- added R-KVPSU1-4: 470K, Resistor_THT:R_Axial_DIN0516_L15.5mm_D5.0mm_P5.08mm_Vertical, F.Cu at (614.1, 88.2)
- added R-KVPSU1-5: 1.5K, Resistor_THT:R_Axial_DIN0516_L15.5mm_D5.0mm_P5.08mm_Vertical, F.Cu at (568.6, 138.1)
- added R-KVPSU1-6: 2R 3W, Resistor_THT:R_Axial_DIN0516_L15.5mm_D5.0mm_P5.08mm_Vertical, F.Cu at (578.9, 125.9)
- added R-KVPSU1-7: 15k 3W, Resistor_THT:R_Axial_DIN0516_L15.5mm_D5.0mm_P5.08mm_Vertical, F.Cu at (614.1, 68.6)
- added R-KVPSU1-8: 22K, Resistor_THT:R_Axial_DIN0516_L15.5mm_D5.0mm_P5.08mm_Vertical, F.Cu at (558.3, 131.5)
- added R-KVPSU1-9: 2R 3W, Resistor_THT:R_Axial_DIN0516_L15.5mm_D5.0mm_P5.08mm_Vertical, F.Cu at (558.3, 125.0)
- added R-KVPSU2-1: 2R 3W, Resistor_THT:R_Axial_DIN0516_L15.5mm_D5.0mm_P5.08mm_Vertical, F.Cu at (610.8, 401.4)
- added R-KVPSU2-2: 700K, Resistor_THT:R_Axial_DIN0516_L15.5mm_D5.0mm_P5.08mm_Vertical, F.Cu at (600.4, 401.4)
- added R-KVPSU2-3: 800K, Resistor_THT:R_Axial_DIN0516_L15.5mm_D5.0mm_P5.08mm_Vertical, F.Cu at (600.4, 407.9)
- added R-KVPSU2-4: .7k, Resistor_THT:R_Axial_DIN0516_L15.5mm_D5.0mm_P5.08mm_Vertical, F.Cu at (651.7, 372.2)
- added RV-KVPSU1-1: 500K WW, Potentiometer_THT:Potentiometer_Piher_PT-10-V05_Vertical, F.Cu at (540.6, 116.3)
- added S1: 7205SYCQE, SamacSys_Parts_m:7205SYCQE, F.Cu at (471.0, 385.7)
- added S2: 7205SYCQE, SamacSys_Parts_m:7205SYCQE, F.Cu at (498.1, 358.0)
- added SW-KEYSW2-1: SW_DPDT_x2, SamacSys_Parts_m:7205SYCQE, F.Cu at (525.2, 344.2)
- added SW-KVPSU1-2: SW_SPST, Connector_PinHeader_2.54mm:PinHeader_1x04_P2.54mm_Vertical, F.Cu at (534.9, 110.2)
- added SW-KVPSU2-2: EHT switch, Connector_PinHeader_2.54mm:PinHeader_1x04_P2.54mm_Vertical, F.Cu at (650.7, 359.0)
- added TR-KVPSU1-1: VARIAC, Connector_PinHeader_2.54mm:PinHeader_1x10_P2.54mm_Vertical, F.Cu at (525.6, 96.4)
- added TR-KVPSU1-2: Transformer_1P_1S, Connector_PinHeader_2.54mm:PinHeader_1x04_P2.54mm_Vertical, F.Cu at (530.2, 110.2)
- added TR-KVPSU1-3: Transformer_1P_4S, Connector_PinHeader_2.54mm:PinHeader_1x10_P2.54mm_Vertical, F.Cu at (554.3, 67.6)
- added TR-KVPSU2-1: VARIAC, Connector_PinHeader_2.54mm:PinHeader_1x10_P2.54mm_Vertical, F.Cu at (591.9, 359.0)
- added TR-KVPSU2-2: Transformer_1P_1S, Connector_PinHeader_2.54mm:PinHeader_1x04_P2.54mm_Vertical, F.Cu at (594.8, 400.4)
- added TR-KVPSU2-3: Transformer_1P_4S, Connector_PinHeader_2.54mm:PinHeader_1x10_P2.54mm_Vertical, F.Cu at (563.1, 387.7)
- added U-KVPSU1-1: VU111, NewValves:Valve_B4+1, F.Cu at (595.7, 105.3)
- added U-KVPSU1-3: CV71, Connector_PinHeader_2.54mm:PinHeader_1x02_P2.54mm_Vertical, F.Cu at (579.8, 109.1)
- added V-KVPSU1-1: VR91, NewValves:Valve_9Loctal, F.Cu at (508.9, 79.7)
- added V-KVPSU1-2: VR91, NewValves:Valve_9Loctal, F.Cu at (508.9, 108.4)
- added V-KVPSU1-3: CV73, NewValves:Valve_9Loctal, F.Cu at (537.6, 79.7)
- added V-KVPSU2-1: VU111, NewValves:Valve_B4+1, F.Cu at (633.3, 396.6)
- added V-KVPSU2-4: CV71, Valve:Valve_Octal, F.Cu at (582.8, 378.6)
- J-KEYSW1-10: value Hs -> CL.13
- J-KEYSW1-2: value CL.4 -> Hs
- J-KEYSW1-3: value CL.3 -> CL.4
- J-KEYSW1-4: value CL.2 -> CL.3
- J-KEYSW1-5: value CL.1 -> CL.2
- J-KEYSW1-6: value CL.0 -> CL.1
- J-KEYSW1-7: value CL.15 -> CL.0
- J-KEYSW1-8: value CL.14 -> CL.15
- J-KEYSW1-9: value CL.13 -> CL.14
- SW-KEYSW1-1: value SW_DPDT_x2 -> SW_Push; footprint SamacSys_Parts_m:7205SYCQE -> Button_Switch_THT:SW_PUSH-12mm
- SW-KEYSW1-2: value SW_Push -> SW_DPDT_x2; footprint Button_Switch_THT:SW_PUSH-12mm -> SamacSys_Parts_m:7205SYCQE
- moved U-CMOSCRT1-4 252.3 mm to (650.4, 230.5)
- moved D-CMOSCRT1-2 238.2 mm to (661.5, 230.5)
- moved R-CMOSCRT1-2 236.5 mm to (673.2, 240.2)
- moved R-ADDER1-35 233.5 mm to (-35.8, 86.5)
- moved D1 226.9 mm to (639.8, 249.9)
- moved C-CMOSCRT1-5 226.5 mm to (674.5, 246.7)
- moved D-CMOSCRT1-7 223.6 mm to (661.5, 234.8)
- moved U-CMOSCRT1-3 213.9 mm to (628.7, 252.4)
- moved C-CMOSCRT1-4 212.1 mm to (673.2, 253.3)
- moved R-CMOSCRT1-7 208.2 mm to (655.1, 251.1)
- moved R-CMOSCRT1-5 208.1 mm to (665.4, 246.7)
- moved R-CRTCCT3-6 204.4 mm to (763.0, 76.9)
- moved R-ADDER1-23 204.4 mm to (164.3, -8.88)
- moved J-KEYSW1-10 201.9 mm to (605.8, 327.3)
- moved J-CMOSCRT1-2 198.8 mm to (605.8, 235.0)
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Connections:
- Fn-KEYSW1-1 pad 3: Net-(Fn-KEYSW1-0-Pad3) -> Net-(Fn-KEYSW1-1-Pad3)
- Fn-KEYSW1-2 pad 3: Net-(Fn-KEYSW1-0-Pad3) -> Net-(Fn-KEYSW1-1-Pad3)
- J-KEYSW1-10 pad 1: Net-(J-KEYSW1-10-Pad1) -> Net-(Fn-KEYSW1-3-Pad2)
- J-KEYSW1-7 pad 1: Net-(Fn-KEYSW1-2-Pad2) -> Net-(J-KEYSW1-7-Pad1)
- J-KEYSW1-9 pad 1: Net-(Fn-KEYSW1-0-Pad2) -> Net-(Fn-KEYSW1-2-Pad2)
- L-KEYSW1-1 pad 2: Net-(J-KEYSW1-5-Pad1) -> Net-(J-KEYSW1-3-Pad1)
- L-KEYSW1-1 pad 3: Net-(Fn-KEYSW1-0-Pad3) -> Net-(Fn-KEYSW1-1-Pad3)
- L-KEYSW1-2 pad 3: Net-(Fn-KEYSW1-0-Pad3) -> Net-(Fn-KEYSW1-1-Pad3)
- L-KEYSW1-3 pad 2: Net-(J-KEYSW1-3-Pad1) -> Net-(J-KEYSW1-5-Pad1)
- L-KEYSW1-3 pad 3: Net-(Fn-KEYSW1-0-Pad3) -> Net-(Fn-KEYSW1-1-Pad3)
- L-KEYSW1-4 pad 2: Net-(J-KEYSW1-2-Pad1) -> Net-(J-KEYSW1-6-Pad1)
- L-KEYSW1-4 pad 3: Net-(Fn-KEYSW1-0-Pad3) -> Net-(Fn-KEYSW1-1-Pad3)
- SW-KEYSW1-1 pad 1: (no net) -> Net-(J-KEYSW1-1-Pad1)
- SW-KEYSW1-1 pad 2: Net-(Fn-KEYSW1-0-Pad3) -> Net-(J-KEYSW1-2-Pad1)
- SW-KEYSW1-2 pad 1: Net-(J-KEYSW1-1-Pad1) -> (no net)
- SW-KEYSW1-2 pad 2: Net-(J-KEYSW1-10-Pad1) -> Net-(Fn-KEYSW1-1-Pad3)
- U-CRTPCIF2-5 pad 8: (no net) -> /CRTPCIF2/Bk1

Commit message: Add L-STAT.
Signed-off-by: John Bradley <flypie@rocketmail.com>
Parts:
- added C-L-STAT-1: 47p, Capacitor_THT:C_Disc_D7.5mm_W5.0mm_P5.00mm, F.Cu at (364.1, 148.9)
- added C-L-STAT-10: 0.1, Capacitor_THT:C_Disc_D7.5mm_W5.0mm_P5.00mm, F.Cu at (338.9, 176.9)
- added C-L-STAT-11: 0.5, Capacitor_THT:C_Disc_D7.5mm_W5.0mm_P5.00mm, F.Cu at (349.2, 163.1)
- added C-L-STAT-13: 0.5, Capacitor_THT:C_Disc_D7.5mm_W5.0mm_P5.00mm, F.Cu at (379.8, 134.3)
- added C-L-STAT-14: 0.5, Capacitor_THT:C_Disc_D7.5mm_W5.0mm_P5.00mm, F.Cu at (332.3, 190.0)
- added C-L-STAT-15: 0.5, Capacitor_THT:C_Disc_D7.5mm_W5.0mm_P5.00mm, F.Cu at (328.5, 183.5)
- added C-L-STAT-2: 100pF, Capacitor_THT:C_Disc_D7.5mm_W5.0mm_P5.00mm, F.Cu at (349.2, 169.7)
- added C-L-STAT-3: 100pF, Capacitor_THT:C_Disc_D7.5mm_W5.0mm_P5.00mm, F.Cu at (379.8, 140.9)
- added C-L-STAT-4: 100pF, Capacitor_THT:C_Disc_D7.5mm_W5.0mm_P5.00mm, F.Cu at (358.3, 162.0)
- added C-L-STAT-5: 0.1, Capacitor_THT:C_Disc_D7.5mm_W5.0mm_P5.00mm, F.Cu at (337.6, 183.5)
- added C-L-STAT-6: 100pF, Capacitor_THT:C_Disc_D7.5mm_W5.0mm_P5.00mm, F.Cu at (322.5, 200.7)
- added C-L-STAT-7: 47pF, Capacitor_THT:C_Disc_D7.5mm_W5.0mm_P5.00mm, F.Cu at (373.2, 147.4)
- added C-L-STAT-8: 2^(n-1)*0.01, Capacitor_THT:C_Disc_D7.5mm_W5.0mm_P5.00mm, F.Cu at (388.9, 134.3)
- added C-L-STAT-9: 0.1, Capacitor_THT:C_Disc_D7.5mm_W5.0mm_P5.00mm, F.Cu at (364.1, 155.4)
- added D-L-STAT-5: EA50, NewValves:Valve_B3G, F.Cu at (333.1, 154.0)
- added D-L-STAT-6: EA50, NewValves:Valve_B3G, F.Cu at (367.3, 111.4)
- added D-L-STAT-7: EA50, NewValves:Valve_B3G, F.Cu at (338.5, 140.2)
- added D-L-STAT-8: EA50, NewValves:Valve_B3G, F.Cu at (297.5, 182.8)
- added D-L-STAT-9: EA50, NewValves:Valve_B3G, F.Cu at (282.6, 182.8)
- added J-L-STAT-1: Cn-1, SamacSys_Parts_l:242431, F.Cu at (339.4, 125.3)
- added J-L-STAT-17: HIGH Voltage., Connector_TE-Connectivity:TE_MATE-N-LOK_1-770970-x_2x04_P4.14mm_Horizontal, F.Cu at (307.2, 151.3)
- added J-L-STAT-2: Cl-N, SamacSys_Parts_l:242431, F.Cu at (224.3, 197.8)
- added J-L-STAT-3: P.n, SamacSys_Parts_l:242431, F.Cu at (278.5, 197.8)
- added J-L-STAT-4: HA, SamacSys_Parts_l:242431, F.Cu at (339.4, 111.5)
- added J-L-STAT-5: HA, SamacSys_Parts_l:242431, F.Cu at (310.6, 140.3)
- added J-L-STAT-6: Cn, SamacSys_Parts_l:242431, F.Cu at (281.9, 169.0)
- added J-L-STAT-7: HS, SamacSys_Parts_l:242431, F.Cu at (251.4, 197.8)
- added R-L-STAT-1: 47K, Resistor_THT:R_Axial_DIN0516_L15.5mm_D5.0mm_P5.08mm_Vertical, F.Cu at (389.2, 114.7)
- added R-L-STAT-10: 330K, Resistor_THT:R_Axial_DIN0516_L15.5mm_D5.0mm_P5.08mm_Vertical, F.Cu at (306.4, 170.9)
- added R-L-STAT-11: 19K, Resistor_THT:R_Axial_DIN0516_L15.5mm_D5.0mm_P5.08mm_Vertical, F.Cu at (303.1, 199.2)
- added R-L-STAT-12: 390K, Resistor_THT:R_Axial_DIN0516_L15.5mm_D5.0mm_P5.08mm_Vertical, F.Cu at (360.4, 135.8)
- added R-L-STAT-13: 390K, Resistor_THT:R_Axial_DIN0516_L15.5mm_D5.0mm_P5.08mm_Vertical, F.Cu at (350.1, 142.3)
- added R-L-STAT-14: 47K 1W, Resistor_THT:R_Axial_DIN0516_L15.5mm_D5.0mm_P5.08mm_Vertical, F.Cu at (374.3, 121.2)
- added R-L-STAT-15: 330K, Resistor_THT:R_Axial_DIN0516_L15.5mm_D5.0mm_P5.08mm_Vertical, F.Cu at (364.0, 127.8)
- added R-L-STAT-16: 47K 1W, Resistor_THT:R_Axial_DIN0516_L15.5mm_D5.0mm_P5.08mm_Vertical, F.Cu at (389.2, 108.1)
- added R-L-STAT-17: 10K, Resistor_THT:R_Axial_DIN0516_L15.5mm_D5.0mm_P5.08mm_Vertical, F.Cu at (378.9, 114.7)
- added R-L-STAT-18: 180K, Resistor_THT:R_Axial_DIN0516_L15.5mm_D5.0mm_P5.08mm_Vertical, F.Cu at (364.0, 121.2)
- added R-L-STAT-19: 330K, Resistor_THT:R_Axial_DIN0516_L15.5mm_D5.0mm_P5.08mm_Vertical, F.Cu at (329.8, 163.8)
- added R-L-STAT-2: 47K, Resistor_THT:R_Axial_DIN0516_L15.5mm_D5.0mm_P5.08mm_Vertical, F.Cu at (319.5, 184.0)
- added R-L-STAT-20: 390K, Resistor_THT:R_Axial_DIN0516_L15.5mm_D5.0mm_P5.08mm_Vertical, F.Cu at (309.1, 177.5)
- added R-L-STAT-21: 19K, Resistor_THT:R_Axial_DIN0516_L15.5mm_D5.0mm_P5.08mm_Vertical, F.Cu at (344.7, 150.0)
- added R-L-STAT-22: 330K, Resistor_THT:R_Axial_DIN0516_L15.5mm_D5.0mm_P5.08mm_Vertical, F.Cu at (316.8, 170.9)
- added R-L-STAT-23: 330K, Resistor_THT:R_Axial_DIN0516_L15.5mm_D5.0mm_P5.08mm_Vertical, F.Cu at (303.1, 192.6)
- added R-L-STAT-24: 1M, Resistor_THT:R_Axial_DIN0516_L15.5mm_D5.0mm_P5.08mm_Vertical, F.Cu at (384.6, 127.8)
- added R-L-STAT-25: 11K 2W, Resistor_THT:R_Axial_DIN0516_L15.5mm_D5.0mm_P5.08mm_Vertical, F.Cu at (319.5, 177.5)
- added R-L-STAT-26: 15K 2W, Resistor_THT:R_Axial_DIN0516_L15.5mm_D5.0mm_P5.08mm_Vertical, F.Cu at (340.2, 170.4)
- added R-L-STAT-27: 33K 2W, Resistor_THT:R_Axial_DIN0516_L15.5mm_D5.0mm_P5.08mm_Vertical, F.Cu at (374.3, 127.8)
- added R-L-STAT-28: 15K 2W, Resistor_THT:R_Axial_DIN0516_L15.5mm_D5.0mm_P5.08mm_Vertical, F.Cu at (370.8, 140.9)
- added R-L-STAT-29: 330K, Resistor_THT:R_Axial_DIN0516_L15.5mm_D5.0mm_P5.08mm_Vertical, F.Cu at (313.4, 197.1)
- added R-L-STAT-3: 330K, Resistor_THT:R_Axial_DIN0516_L15.5mm_D5.0mm_P5.08mm_Vertical, F.Cu at (313.4, 190.6)
- added R-L-STAT-30: 100K, Resistor_THT:R_Axial_DIN0516_L15.5mm_D5.0mm_P5.08mm_Vertical, F.Cu at (329.8, 176.9)
- added R-L-STAT-31: 470, Resistor_THT:R_Axial_DIN0516_L15.5mm_D5.0mm_P5.08mm_Vertical, F.Cu at (370.8, 134.3)
- added R-L-STAT-32: 9K 6W, Resistor_THT:R_Axial_DIN0516_L15.5mm_D5.0mm_P5.08mm_Vertical, F.Cu at (355.0, 148.9)
- added R-L-STAT-33: 100K, Resistor_THT:R_Axial_DIN0516_L15.5mm_D5.0mm_P5.08mm_Vertical, F.Cu at (340.2, 163.8)
- added R-L-STAT-34: 270K, Resistor_THT:R_Axial_DIN0516_L15.5mm_D5.0mm_P5.08mm_Vertical, F.Cu at (360.4, 142.3)
- added R-L-STAT-35: R, Resistor_THT:R_Axial_DIN0516_L15.5mm_D5.0mm_P5.08mm_Vertical, F.Cu at (384.6, 121.2)
- added R-L-STAT-4: 560K, Resistor_THT:R_Axial_DIN0516_L15.5mm_D5.0mm_P5.08mm_Vertical, F.Cu at (350.1, 135.8)
- added R-L-STAT-5: 10K, Resistor_THT:R_Axial_DIN0516_L15.5mm_D5.0mm_P5.08mm_Vertical, F.Cu at (344.7, 156.6)
- added R-L-STAT-6: 47K 1W, Resistor_THT:R_Axial_DIN0516_L15.5mm_D5.0mm_P5.08mm_Vertical, F.Cu at (355.0, 155.4)
- added R-L-STAT-7: 47K 1W, Resistor_THT:R_Axial_DIN0516_L15.5mm_D5.0mm_P5.08mm_Vertical, F.Cu at (309.1, 184.0)
- added R-L-STAT-8: 390K, Resistor_THT:R_Axial_DIN0516_L15.5mm_D5.0mm_P5.08mm_Vertical, F.Cu at (378.9, 108.1)
- added R-L-STAT-9: 330K, Resistor_THT:R_Axial_DIN0516_L15.5mm_D5.0mm_P5.08mm_Vertical, F.Cu at (329.8, 170.4)
- added RV-L-STAT-36: R', Potentiometer_THT:3362H1103LF, F.Cu at (325.4, 192.4)
- added V-L-STAT-1: 6SN7GT, Valve:Valve_Octal, F.Cu at (269.3, 184.4)
- added V-L-STAT-2: 6SN7GT, Valve:Valve_Octal, F.Cu at (298.1, 126.9)
- added V-L-STAT-3: VR91, NewValves:Valve_9Loctal, F.Cu at (319.2, 119.2)
- added V-L-STAT-4: VR91, NewValves:Valve_9Loctal, F.Cu at (261.7, 148.0)
- added V-L-STAT-5: VR91, NewValves:Valve_9Loctal, F.Cu at (232.9, 176.8)
- added V-L-STAT-6: VR91, NewValves:Valve_9Loctal, F.Cu at (261.7, 119.2)
- added V-L-STAT-7: VR91, NewValves:Valve_9Loctal, F.Cu at (232.9, 119.2)
- added V-L-STAT-8: VR91, NewValves:Valve_9Loctal, F.Cu at (290.5, 148.0)
- added V-L-STAT-9: VR91, NewValves:Valve_9Loctal, F.Cu at (232.9, 148.0)
- moved R-CTRLGATE-9 624.5 mm to (31.9, 408.8)
- moved R-CTRLGATE-4 598.6 mm to (73.2, 407.6)
- moved R-CTRLGATE-6 592.0 mm to (109.5, 406.9)
- moved J-CTRLGATE-7 578.4 mm to (63.2, 397.2)
- moved J-CMOSCRT2-1 561.5 mm to (641.0, 89.0)
- moved D-CMOSCRT2-14 558.8 mm to (685.9, 88.7)
- moved D-CMOSCRT2-12 555.2 mm to (664.6, 106.4)
- moved R-CTRLGATE-8 552.0 mm to (42.2, 408.8)
- moved R-CTRLGATE-13 550.4 mm to (124.4, 403.3)
- moved R-CMOSCRT2-52 548.6 mm to (701.2, 91.6)
- moved J-CTRLGATE-5 546.1 mm to (119.0, 353.5)
- moved J-CTRLGATE-6 546.1 mm to (91.9, 367.3)
- moved D-CMOSCRT2-13 538.5 mm to (653.8, 125.8)
- moved C-CTRLGATE-6 536.6 mm to (133.4, 403.3)
- moved D-CTRLGATE-5 532.6 mm to (112.7, 397.1)
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
Commit message: Add Monicct & MonSW. KiCAD auto changed some of the rest.
Signed-off-by: John Bradley <flypie@rocketmail.com>
Parts:
- removed J-ADDER1-16: HIGH Voltage., Connector_TE-Connectivity:TE_MATE-N-LOK_1-770970-x_2x04_P4.14mm_Horizontal
- added C-MONICCT-1: 0.5 4kV, Capacitor_THT:C_Disc_D7.5mm_W5.0mm_P5.00mm, F.Cu at (829.2, 161.9)
- added C-MONICCT-2: 0.1, Capacitor_THT:C_Disc_D7.5mm_W5.0mm_P5.00mm, F.Cu at (814.5, 168.4)
- added C-MONICCT-3: 0.1, Capacitor_THT:C_Disc_D7.5mm_W5.0mm_P5.00mm, F.Cu at (839.5, 152.7)
- added C-MONICCT-4: 0.1 350V, Capacitor_THT:C_Disc_D7.5mm_W5.0mm_P5.00mm, F.Cu at (823.6, 168.4)
- added C-MONICCT-5: 0.1 350V, Capacitor_THT:C_Disc_D7.5mm_W5.0mm_P5.00mm, F.Cu at (814.5, 175.0)
- added C-MONICCT-7: 0.25 4kv, Capacitor_THT:C_Disc_D7.5mm_W5.0mm_P5.00mm, F.Cu at (847.0, 140.1)
- added C-MONSW-1: 1000, Capacitor_THT:C_Disc_D7.5mm_W5.0mm_P5.00mm, F.Cu at (201.0, 184.2)
- added C-MONSW-10: 0.1, Capacitor_THT:C_Disc_D7.5mm_W5.0mm_P5.00mm, F.Cu at (162.3, 213.0)
- added C-MONSW-11: 0.5, Capacitor_THT:C_Disc_D7.5mm_W5.0mm_P5.00mm, F.Cu at (205.5, 169.7)
- added C-MONSW-2: 0.1, Capacitor_THT:C_Disc_D7.5mm_W5.0mm_P5.00mm, F.Cu at (147.5, 233.2)
- added C-MONSW-3: 1000, Capacitor_THT:C_Disc_D7.5mm_W5.0mm_P5.00mm, F.Cu at (205.5, 176.3)
- added C-MONSW-4: 0.5, Capacitor_THT:C_Disc_D7.5mm_W5.0mm_P5.00mm, F.Cu at (182.9, 197.4)
- added C-MONSW-5: 0.5, Capacitor_THT:C_Disc_D7.5mm_W5.0mm_P5.00mm, F.Cu at (192.0, 190.8)
- added C-MONSW-6: 0.1, Capacitor_THT:C_Disc_D7.5mm_W5.0mm_P5.00mm, F.Cu at (141.1, 241.1)
- added C-MONSW-7: 0.5, Capacitor_THT:C_Disc_D7.5mm_W5.0mm_P5.00mm, F.Cu at (172.6, 206.9)
- added C-MONSW-8: 0.5, Capacitor_THT:C_Disc_D7.5mm_W5.0mm_P5.00mm, F.Cu at (182.9, 190.8)
- added C-MONSW-9: 1000, Capacitor_THT:C_Disc_D7.5mm_W5.0mm_P5.00mm, F.Cu at (157.9, 220.1)
- added D-MONICCT-1: EA50, NewValves:Valve_B3G, F.Cu at (851.6, 114.5)
- added D-MONSW-1: EA50, NewValves:Valve_B3G, F.Cu at (118.0, 218.1)
- added D-MONSW-2: EA50, NewValves:Valve_B3G, F.Cu at (184.9, 174.4)
- added D-MONSW-3: EA50, NewValves:Valve_B3G, F.Cu at (202.6, 146.8)
- added J-CRTCCT5-16: HIGH Voltage., Connector_TE-Connectivity:TE_MATE-N-LOK_1-770970-x_2x04_P4.14mm_Horizontal, F.Cu at (594.7, 369.8)
- added J-MONICCT-1: STOP.LAMP, SamacSys_Parts_l:242431, F.Cu at (796.6, 142.2)
- added J-MONICCT-16: HIGH Voltage., Connector_TE-Connectivity:TE_MATE-N-LOK_1-770970-x_2x04_P4.14mm_Horizontal, F.Cu at (793.1, 167.1)
- added J-MONICCT-2: Y2, SamacSys_Parts_l:242431, F.Cu at (823.7, 114.6)
- added J-MONICCT-3: A.Y1, SamacSys_Parts_l:242431, F.Cu at (796.6, 128.4)
- added J-MONICCT-4: A.X2, SamacSys_Parts_l:242431, F.Cu at (796.6, 114.6)
- added J-MONICCT-5: A.X1, SamacSys_Parts_l:242431, F.Cu at (796.6, 156.1)
- added J-MONICCT-6: +300, SamacSys_Parts_l:242431, F.Cu at (823.7, 142.2)
- added J-MONICCT-7: M.GRID, SamacSys_Parts_l:242431, F.Cu at (823.7, 128.4)
- added J-MONSW-5: HIGH Voltage., Connector_TE-Connectivity:TE_MATE-N-LOK_1-770970-x_2x04_P4.14mm_Horizontal, F.Cu at (140.9, 200.5)
- added J-MONSW1: C.GRID, SamacSys_Parts_l:242431, F.Cu at (118.9, 189.4)
- added J-MONSW10: MON.A, SamacSys_Parts_l:242431, F.Cu at (147.7, 160.7)
- added J-MONSW11: MON.A, SamacSys_Parts_l:242431, F.Cu at (86.8, 233.2)
- added J-MONSW12: MON.C, SamacSys_Parts_l:242431, F.Cu at (147.7, 146.8)
- added J-MONSW13: MON.C, SamacSys_Parts_l:242431, F.Cu at (118.9, 175.6)
- added J-MONSW14: SUP.ACT.LN, SamacSys_Parts_l:242431, F.Cu at (90.1, 204.4)
- added J-MONSW15: SUP.ACT.LN, SamacSys_Parts_l:242431, F.Cu at (59.7, 233.2)
- added J-MONSW2: A.GRID, SamacSys_Parts_l:242431, F.Cu at (90.1, 218.2)
- added J-MONSW3: S.GRID, SamacSys_Parts_l:242431, F.Cu at (117.2, 204.4)
- added J-MONSW4: B, SamacSys_Parts_l:242431, F.Cu at (146.0, 175.6)
- added J-MONSW5: MON.S, SamacSys_Parts_l:242431, F.Cu at (174.8, 146.8)
- added J-MONSW6: M, SamacSys_Parts_l:242431, F.Cu at (113.9, 232.0)
- added J-MONSW7: KM.cmn, SamacSys_Parts_l:242431, F.Cu at (174.8, 160.7)
- added J-MONSW8: KM.cmn, SamacSys_Parts_l:242431, F.Cu at (146.0, 189.4)
- added J-MONSW9: MON.S, SamacSys_Parts_l:242431, F.Cu at (32.6, 233.2)
- added R-MONICCT-1: 1980K, Resistor_THT:R_Axial_DIN0516_L15.5mm_D5.0mm_P5.08mm_Vertical, F.Cu at (737.2, 178.4)
- added R-MONICCT-2: 1K, Resistor_THT:R_Axial_DIN0516_L15.5mm_D5.0mm_P5.08mm_Vertical, F.Cu at (747.6, 178.4)
- added R-MONICCT-3: 1K, Resistor_THT:R_Axial_DIN0516_L15.5mm_D5.0mm_P5.08mm_Vertical, F.Cu at (757.9, 178.4)
- added R-MONICCT-4: 470K, Resistor_THT:R_Axial_DIN0516_L15.5mm_D5.0mm_P5.08mm_Vertical, F.Cu at (768.2, 178.4)
- added R-MONICCT-5: 270K, Resistor_THT:R_Axial_DIN0516_L15.5mm_D5.0mm_P5.08mm_Vertical, F.Cu at (778.6, 178.4)
- added R-MONICCT-6: 2M2, Resistor_THT:R_Axial_DIN0516_L15.5mm_D5.0mm_P5.08mm_Vertical, F.Cu at (848.3, 124.3)
- added R-MONICCT-7: 22K, Resistor_THT:R_Axial_DIN0516_L15.5mm_D5.0mm_P5.08mm_Vertical, F.Cu at (726.9, 178.4)
- added R-MONICCT-8: 2R 3W, Resistor_THT:R_Axial_DIN0516_L15.5mm_D5.0mm_P5.08mm_Vertical, F.Cu at (821.2, 152.7)
- added R-MONSW-1: R 2W, Resistor_THT:R_Axial_DIN0516_L15.5mm_D5.0mm_P5.08mm_Vertical, F.Cu at (173.8, 193.8)
- added R-MONSW-10: 33K 2W, Resistor_THT:R_Axial_DIN0516_L15.5mm_D5.0mm_P5.08mm_Vertical, F.Cu at (199.3, 163.2)
- added R-MONSW-11: 1M, Resistor_THT:R_Axial_DIN0516_L15.5mm_D5.0mm_P5.08mm_Vertical, F.Cu at (163.5, 199.9)
- added R-MONSW-12: 10M, Resistor_THT:R_Axial_DIN0516_L15.5mm_D5.0mm_P5.08mm_Vertical, F.Cu at (170.6, 187.2)
- added R-MONSW-13: 10M, Resistor_THT:R_Axial_DIN0516_L15.5mm_D5.0mm_P5.08mm_Vertical, F.Cu at (199.3, 156.6)
- added R-MONSW-14: 4.7K 6W, Resistor_THT:R_Axial_DIN0516_L15.5mm_D5.0mm_P5.08mm_Vertical, F.Cu at (181.6, 184.3)
- added R-MONSW-15: 330K, Resistor_THT:R_Axial_DIN0516_L15.5mm_D5.0mm_P5.08mm_Vertical, F.Cu at (173.8, 200.3)
- added R-MONSW-16: R, Resistor_THT:R_Axial_DIN0516_L15.5mm_D5.0mm_P5.08mm_Vertical, F.Cu at (111.4, 242.5)
- added R-MONSW-17: 4.7K 6W, Resistor_THT:R_Axial_DIN0516_L15.5mm_D5.0mm_P5.08mm_Vertical, F.Cu at (129.6, 214.9)
- added R-MONSW-18: 47K, Resistor_THT:R_Axial_DIN0516_L15.5mm_D5.0mm_P5.08mm_Vertical, F.Cu at (138.5, 221.4)
- added R-MONSW-19: 47K, Resistor_THT:R_Axial_DIN0516_L15.5mm_D5.0mm_P5.08mm_Vertical, F.Cu at (148.8, 226.7)
- added R-MONSW-2: 33K 2W, Resistor_THT:R_Axial_DIN0516_L15.5mm_D5.0mm_P5.08mm_Vertical, F.Cu at (196.5, 177.7)
- added R-MONSW-20: R, Resistor_THT:R_Axial_DIN0516_L15.5mm_D5.0mm_P5.08mm_Vertical, F.Cu at (121.7, 242.5)
- added R-MONSW-3: 1M, Resistor_THT:R_Axial_DIN0516_L15.5mm_D5.0mm_P5.08mm_Vertical, F.Cu at (138.5, 234.5)
- added R-MONSW-4: 1K, Resistor_THT:R_Axial_DIN0516_L15.5mm_D5.0mm_P5.08mm_Vertical, F.Cu at (191.9, 184.3)
- added R-MONSW-5: R 2W, Resistor_THT:R_Axial_DIN0516_L15.5mm_D5.0mm_P5.08mm_Vertical, F.Cu at (132.0, 242.5)
- added R-MONSW-6: 33K 2W, Resistor_THT:R_Axial_DIN0516_L15.5mm_D5.0mm_P5.08mm_Vertical, F.Cu at (163.5, 206.5)
- added R-MONSW-7: 1M, Resistor_THT:R_Axial_DIN0516_L15.5mm_D5.0mm_P5.08mm_Vertical, F.Cu at (148.8, 220.1)
- added R-MONSW-8: 15K 3W, Resistor_THT:R_Axial_DIN0516_L15.5mm_D5.0mm_P5.08mm_Vertical, F.Cu at (138.5, 228.0)
- added R-MONSW-9: R 2W, Resistor_THT:R_Axial_DIN0516_L15.5mm_D5.0mm_P5.08mm_Vertical, F.Cu at (196.5, 171.1)
- added RV-MONICCT-1: 500K, Potentiometer_THT:Potentiometer_Bourns_3339P_Vertical_HandSoldering, F.Cu at (849.6, 134.7)
- added RV-MONICCT-2: 100K, Potentiometer_THT:Potentiometer_Bourns_3339P_Vertical_HandSoldering, F.Cu at (832.8, 156.5)
- added RV-MONICCT-3: 100K, Potentiometer_THT:Potentiometer_Bourns_3339P_Vertical_HandSoldering, F.Cu at (822.5, 163.1)
- added SW-MONSW-1: SW-MONSW-1, SamacSys_Parts_l:M2011SS1W03, F.Cu at (176.8, 180.6)
- added SW1: SW_Push, Connector_PinHeader_2.54mm:PinHeader_1x02_P2.54mm_Vertical, F.Cu at (128.6, 220.5)
- added SW2: SW_Push, Connector_PinHeader_2.54mm:PinHeader_1x02_P2.54mm_Vertical, F.Cu at (208.7, 155.7)
- added SW3: SW_Push, Connector_PinHeader_2.54mm:PinHeader_1x02_P2.54mm_Vertical, F.Cu at (183.2, 203.0)
- added SW4: SW_Push, Connector_PinHeader_2.54mm:PinHeader_1x02_P2.54mm_Vertical, F.Cu at (158.2, 225.7)
- added SW5: SW_Push, Connector_PinHeader_2.54mm:PinHeader_1x02_P2.54mm_Vertical, F.Cu at (167.2, 218.6)
- added V-MONICCT-1: VCR97, NewValves:B12D, F.Cu at (757.2, 141.5)
- added V-MONSW-1: VR91, NewValves:Valve_9Loctal, F.Cu at (41.2, 212.1)
- added V-MONSW-2: CV173, NewValves:Valve_9Loctal, F.Cu at (41.2, 154.6)
- added V-MONSW-3: VR91, NewValves:Valve_9Loctal, F.Cu at (98.7, 183.4)
- added V-MONSW-4: VR91, NewValves:Valve_9Loctal, F.Cu at (70.0, 212.1)
- added V-MONSW-5: VR91, NewValves:Valve_9Loctal, F.Cu at (98.7, 154.6)
- added V-MONSW-6: VR91, NewValves:Valve_9Loctal, F.Cu at (70.0, 183.4)
- added V-MONSW-7: VR91, NewValves:Valve_9Loctal, F.Cu at (41.2, 183.4)
- added V-MONSW-8: CV173, NewValves:Valve_9Loctal, F.Cu at (70.0, 154.6)
- added V-MONSW-?=7: VR91, NewValves:Valve_9Loctal, F.Cu at (127.5, 154.6)
- moved C-ACCGATE-1 627.1 mm to (155.4, 419.6)
- moved C-ACCGATE-6 572.4 mm to (165.8, 413.1)
- moved C-ACCGATE-2 555.3 mm to (134.3, 447.3)
- moved C-ACCGATE-4 555.3 mm to (190.0, 392.5)
- moved C-ACCGATE-7 555.3 mm to (134.8, 440.7)
- moved D-ACCGATE-1 555.3 mm to (129.0, 430.9)
- moved D-ACCGATE-2 555.3 mm to (145.1, 403.2)
- moved D-ACCGATE-3 555.3 mm to (78.0, 448.1)
- moved D-ACCGATE-4 555.3 mm to (33.4, 448.1)
- moved D-ACCGATE-5 555.3 mm to (48.2, 448.1)
- moved D-ACCGATE-6 555.3 mm to (63.1, 448.1)
- moved D-ACCGATE-7 555.3 mm to (92.9, 445.8)
- moved D-ACCGATE-8 555.3 mm to (145.1, 416.4)
- moved J-ACCGATE-10 555.3 mm to (118.9, 361.8)
- moved J-ACCGATE-11 555.3 mm to (117.2, 403.3)
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Connections:
- D-CRTCCT4-1 pad 1: (no net) -> /CRTCCT4/Heater-6.3V
- D-CRTCCT4-1 pad 2: (no net) -> /CRTCCT4/S.EHT(800-1400V)
- D-CRTCCT4-1 pad 3: (no net) -> /CRTCCT4/Heater-GND
- D-CRTCCT4-1 pad 4: (no net) -> Net-(C-CRTCCT4-7-Pad2)
- D-CRTCCT5-1 pad 1: (no net) -> /CRTCCT5/Heater-6.3V
- D-CRTCCT5-1 pad 2: (no net) -> /CRTCCT5/S.EHT(800-1400V)
- D-CRTCCT5-1 pad 3: (no net) -> /CRTCCT5/Heater-GND
- D-CRTCCT5-1 pad 4: (no net) -> Net-(C-CRTCCT5-7-Pad2)

Commit message: Finish KEYSW2/ Add extra Symbols for switches.
Signed-off-by: John Bradley <flypie@rocketmail.com>
Parts:
- removed Fn-KEYSW2-1, Fn-KEYSW2-2, Fn-KEYSW2-3, L-KEYSW2-1, L-KEYSW2-10, L-KEYSW2-11, L-KEYSW2-12, L-KEYSW2-13, L-KEYSW2-14, L-KEYSW2-15, L-KEYSW2-2, L-KEYSW2-3, L-KEYSW2-4, L-KEYSW2-5, L-KEYSW2-8, L-KEYSW2-9: SW_SPDT, SamacSys_Parts_m:A101SYCQ04
- removed J-KEYSW2-7: CL.14, SamacSys_Parts_l:242431
- removed J-KEYSW2-8: CL.13, SamacSys_Parts_l:242431
- removed L-KEYSW2-16: SW_Push_Dual, Connector_PinHeader_2.54mm:PinHeader_1x04_P2.54mm_Vertical
- removed S1, S2: 7205SYCQE, SamacSys_Parts_m:7205SYCQE
- added SW-KEYSW2-16: SW_Double_Acting_Push, Connector_PinHeader_2.54mm:PinHeader_1x04_P2.54mm_Vertical, F.Cu at (751.8, 436.3)
- added SW-KEYSW2-2: SW_QPDT, Connector_PinHeader_2.54mm:PinHeader_1x12_P2.54mm_Vertical, F.Cu at (674.1, 436.3)
- added SW-KEYSW2-3: 7205SYCQE, SamacSys_Parts_m:7205SYCQE, F.Cu at (726.2, 474.2)
- added SW-KEYSW2-4: SW_Push_DPDT, Connector_PinHeader_2.54mm:PinHeader_1x06_P2.54mm_Vertical, F.Cu at (737.6, 436.3)
- added SW-KEYSW2-5: SW_Push_DPDT, Connector_PinHeader_2.54mm:PinHeader_1x06_P2.54mm_Vertical, F.Cu at (733.0, 436.3)
- added SW10: SW_Push, Connector_PinHeader_2.54mm:PinHeader_1x02_P2.54mm_Vertical, F.Cu at (737.6, 453.6)
- added SW6: SW_Push, Connector_PinHeader_2.54mm:PinHeader_1x02_P2.54mm_Vertical, F.Cu at (738.2, 467.1)
- added SW7: SW_Push, Connector_PinHeader_2.54mm:PinHeader_1x02_P2.54mm_Vertical, F.Cu at (733.0, 453.6)
- added SW8: SW_Push, Connector_PinHeader_2.54mm:PinHeader_1x02_P2.54mm_Vertical, F.Cu at (751.8, 448.5)
- added SW9: SW_Push, Connector_PinHeader_2.54mm:PinHeader_1x02_P2.54mm_Vertical, F.Cu at (717.2, 477.8)
- J-KEYSW2-1: value CL.4 -> KM.cmn
- J-KEYSW2-2: value CL.3 -> B
- J-KEYSW2-3: value CL.2 -> M
- J-KEYSW2-4: value CL.1 -> MON.S
- J-KEYSW2-5: value CL.0 -> MON.A
- J-KEYSW2-6: value CL.15 -> MON.C
- R-KEYSW2-2: value 47K -> 100K
- SW-KEYSW2-1: value SW_DPDT_x2 -> SW_QPDT; footprint SamacSys_Parts_m:7205SYCQE -> Connector_PinHeader_2.54mm:PinHeader_1x12_P2.54mm_Vertical
- moved C-CMOSCRT1-2 486.8 mm to (275.3, 502.1)
- moved C-CMOSCRT1-4 486.8 mm to (295.6, 488.9)
- moved C-CMOSCRT1-5 486.8 mm to (308.3, 475.8)
- moved C-CMOSCRT1-6 486.8 mm to (295.6, 482.4)
- moved D-CMOSCRT1-8 486.8 mm to (245.4, 509.4)
- moved D-CMOSCRT1-9 486.8 mm to (250.9, 502.6)
- moved R-CMOSCRT1-1 486.8 mm to (273.9, 495.5)
- moved R-CMOSCRT1-10 486.8 mm to (290.1, 473.6)
- moved R-CMOSCRT1-6 486.8 mm to (308.3, 462.7)
- moved U-CMOSCRT1-3 486.8 mm to (220.4, 494.5)
- moved U-CMOSCRT1-4 486.8 mm to (209.5, 494.5)
- moved U-CMOSCRT1-5 486.8 mm to (236.6, 480.7)
- moved C-CMOSCRT1-3 486.8 mm to (269.8, 508.6)
- moved C-CMOSCRT1-7 486.8 mm to (309.6, 469.3)
- moved D-CMOSCRT1-4 486.8 mm to (274.8, 472.5)
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Connections:
- D-CRTCCT5-1 pad 2: /CRTCCT5/S.EHT(800-1400V) -> (no net)
- J-KEYSW2-1 pad 1: (no net) -> Net-(J-KEYSW2-1-Pad1)
- J-KEYSW2-2 pad 1: (no net) -> Net-(J-KEYSW2-2-Pad1)
- J-KEYSW2-3 pad 1: (no net) -> Net-(J-KEYSW2-3-Pad1)
- J-KEYSW2-4 pad 1: (no net) -> Net-(J-KEYSW2-4-Pad1)
- J-KEYSW2-5 pad 1: (no net) -> Net-(J-KEYSW2-5-Pad1)
- L-KEYSW2-6 pad 1: (no net) -> /KEYSW2/AC.ERASE
- L-KEYSW2-6 pad 2: (no net) -> /KEYSW2/C.ERASE
- L-KEYSW2-6 pad 3: (no net) -> /KEYSW2/-65v
- L-KEYSW2-7 pad 1: (no net) -> /KEYSW2/AC.ERASE
- L-KEYSW2-7 pad 3: (no net) -> /KEYSW2/-65v
- R-KEYSW2-1 pad 1: Net-(L-KEYSW2-3-Pad2) -> /KEYSW2/PC.Read
- R-KEYSW2-1 pad 2: Net-(L-KEYSW2-1-Pad1) -> Net-(R-KEYSW2-1-Pad2)
- R-KEYSW2-2 pad 1: Net-(L-KEYSW2-10-Pad2) -> /KEYSW2/-65v
- R-KEYSW2-2 pad 2: Net-(L-KEYSW2-8-Pad1) -> /KEYSW2/C.ERASE
- SW-KEYSW2-1 pad 2: Net-(Fn-KEYSW2-1-Pad3) -> (no net)
- SW-KEYSW2-1 pad 3: (no net) -> /KEYSW2/PC.Read
- SW-KEYSW2-1 pad 5: (no net) -> Net-(R-KEYSW2-1-Pad2)
- SW-KEYSW2-1 pad 6: (no net) -> /KEYSW2/-65v
