File: KiCAD/SSEMD.kicad_pcb (KiCad board)
At the start: 2 copper layers, 1376 parts, among them SW1 SW_Push, SW10 SW_Push, SW2 SW_Push, SW3 SW_Push, SW4 SW_Push, SW5 SW_Push, SW6 SW_Push, SW7 SW_Push, SW8 SW_Push, SW9 SW_Push, U1 L78L05_TO92

Commit message: Finish powrctl6b
Likely wrong bit of it I didn't understand other bits seem wrong inthe orginal.



Signed-off-by: John Bradley <flypie@rocketmail.com>
Parts:
- added CB-POWRCTL6b-1: RS_63C_16, Connector_PinHeader_2.54mm:PinHeader_1x06_P2.54mm_Vertical, F.Cu at (719.7, 86.3)
- added CR-POWRCTL6b-1: DILA-22, Connector_PinHeader_2.54mm:PinHeader_1x10_P2.54mm_Vertical, F.Cu at (668.6, 113.8)
- added CR-POWRCTL6b-4: DILA-22, Connector_PinHeader_2.54mm:PinHeader_1x10_P2.54mm_Vertical, F.Cu at (673.2, 86.3)
- added CR-POWRCTL6b-A2: DILA-40, Connector_PinHeader_2.54mm:PinHeader_1x10_P2.54mm_Vertical, F.Cu at (687.2, 86.3)
- added CR-POWRCTL6b-A3: DILA-40, Connector_PinHeader_2.54mm:PinHeader_1x10_P2.54mm_Vertical, F.Cu at (682.5, 86.3)
- added CR-POWRCTL6b-B2: DILA-XHI10, Connector_PinHeader_2.54mm:PinHeader_1x10_P2.54mm_Vertical, F.Cu at (677.9, 86.3)
- added CR-POWRCTL6b-B3: DILA-XHI01, Connector_PinHeader_2.54mm:PinHeader_1x10_P2.54mm_Vertical, F.Cu at (668.6, 86.3)
- added D-POWRCTL6b-1: D_Schottky 10A 150V, Package_TO_SOT_THT:TO-46-2, F.Cu at (756.8, 125.5)
- added D-POWRCTL6b-10: D_Schottky 10A 150V, Package_TO_SOT_THT:TO-46-2, F.Cu at (789.0, 105.5)
- added D-POWRCTL6b-11: D_Schottky 10A 150V, Package_TO_SOT_THT:TO-46-2, F.Cu at (746.0, 142.9)
- added D-POWRCTL6b-12: D_Schottky 10A 150V, Package_TO_SOT_THT:TO-46-2, F.Cu at (746.0, 150.6)
- added D-POWRCTL6b-13: D_Schottky 10A 150V, Package_TO_SOT_THT:TO-46-2, F.Cu at (775.6, 114.5)
- added D-POWRCTL6b-14: D_Schottky 10A 150V, Package_TO_SOT_THT:TO-46-2, F.Cu at (764.6, 123.0)
- added D-POWRCTL6b-15: D_Schottky 10A 150V, Package_TO_SOT_THT:TO-46-2, F.Cu at (735.9, 153.9)
- added D-POWRCTL6b-16: D_Schottky 10A 150V, Package_TO_SOT_THT:TO-46-2, F.Cu at (767.9, 114.5)
- added D-POWRCTL6b-17: D_Schottky 10A 150V, Package_TO_SOT_THT:TO-46-2, F.Cu at (773.6, 106.8)
- added D-POWRCTL6b-18: D_Schottky 10A 150V, Package_TO_SOT_THT:TO-46-2, F.Cu at (781.3, 105.5)
- added D-POWRCTL6b-2: D_Schottky 10A 150V, Package_TO_SOT_THT:TO-46-2, F.Cu at (728.2, 153.9)
- added D-POWRCTL6b-3: D_Schottky 10A 150V, Package_TO_SOT_THT:TO-46-2, F.Cu at (738.2, 144.5)
- added D-POWRCTL6b-4: D_Schottky 10A 150V, Package_TO_SOT_THT:TO-46-2, F.Cu at (744.6, 135.2)
- added D-POWRCTL6b-5: D_Schottky 10A 150V, Package_TO_SOT_THT:TO-46-2, F.Cu at (784.7, 97.8)
- added D-POWRCTL6b-6: D_Schottky 10A 150V, Package_TO_SOT_THT:TO-46-2, F.Cu at (792.5, 97.8)
- added D-POWRCTL6b-7: D_Schottky 10A 150V, Package_TO_SOT_THT:TO-46-2, F.Cu at (752.4, 135.2)
- added D-POWRCTL6b-8: D_Schottky 10A 150V, Package_TO_SOT_THT:TO-46-2, F.Cu at (753.7, 142.9)
- added D-POWRCTL6b-9: D_Schottky 10A 150V, Package_TO_SOT_THT:TO-46-2, F.Cu at (760.1, 133.2)
- added F-POWRCTL6b-1: 1A, Connector_PinHeader_2.54mm:PinHeader_1x02_P2.54mm_Vertical, F.Cu at (790.4, 118.7)
- added F-POWRCTL6b-2: 4A, Connector_PinHeader_2.54mm:PinHeader_1x02_P2.54mm_Vertical, F.Cu at (771.8, 120.5)
- added F-POWRCTL6b-3: Fuse, Connector_PinHeader_2.54mm:PinHeader_1x02_P2.54mm_Vertical, F.Cu at (782.9, 111.5)
- added F-POWRCTL6b-4: Fuse, Connector_PinHeader_2.54mm:PinHeader_1x02_P2.54mm_Vertical, F.Cu at (787.5, 111.5)
- added F-POWRCTL6b-5: Fuse, Connector_PinHeader_2.54mm:PinHeader_1x02_P2.54mm_Vertical, F.Cu at (776.5, 120.5)
- added J-POWRCTL6b-1: L, TerminalBlock_MetzConnect:TerminalBlock_MetzConnect_360271_1x01_Horizontal_ScrewM3.0_Boxed, F.Cu at (743.9, 107.4)
- added J-POWRCTL6b-10: 3, TerminalBlock_MetzConnect:TerminalBlock_MetzConnect_360271_1x01_Horizontal_ScrewM3.0_Boxed, F.Cu at (732.8, 126.1)
- added J-POWRCTL6b-11: 3, TerminalBlock_MetzConnect:TerminalBlock_MetzConnect_360271_1x01_Horizontal_ScrewM3.0_Boxed, F.Cu at (754.9, 116.7)
- added J-POWRCTL6b-12: Conn_WallSocket, Connector_PinHeader_2.54mm:PinHeader_1x02_P2.54mm_Vertical, F.Cu at (771.8, 127.7)
- added J-POWRCTL6b-13: 5, TerminalBlock_MetzConnect:TerminalBlock_MetzConnect_360271_1x01_Horizontal_ScrewM3.0_Boxed, F.Cu at (731.7, 135.4)
- added J-POWRCTL6b-14: 4, TerminalBlock_MetzConnect:TerminalBlock_MetzConnect_360271_1x01_Horizontal_ScrewM3.0_Boxed, F.Cu at (771.8, 98.0)
- added J-POWRCTL6b-15: 6, TerminalBlock_MetzConnect:TerminalBlock_MetzConnect_360271_1x01_Horizontal_ScrewM3.0_Boxed, F.Cu at (720.6, 132.3)
- added J-POWRCTL6b-16: 7, TerminalBlock_MetzConnect:TerminalBlock_MetzConnect_360271_1x01_Horizontal_ScrewM3.0_Boxed, F.Cu at (754.9, 107.4)
- added J-POWRCTL6b-17: 10, TerminalBlock_MetzConnect:TerminalBlock_MetzConnect_360271_1x01_Horizontal_ScrewM3.0_Boxed, F.Cu at (709.6, 151.0)
- added J-POWRCTL6b-18: 5, TerminalBlock_MetzConnect:TerminalBlock_MetzConnect_360271_1x01_Horizontal_ScrewM3.0_Boxed, F.Cu at (710.7, 123.0)
- added J-POWRCTL6b-19: 7, TerminalBlock_MetzConnect:TerminalBlock_MetzConnect_360271_1x01_Horizontal_ScrewM3.0_Boxed, F.Cu at (771.8, 88.7)
- added J-POWRCTL6b-2: L, TerminalBlock_MetzConnect:TerminalBlock_MetzConnect_360271_1x01_Horizontal_ScrewM3.0_Boxed, F.Cu at (698.5, 151.0)
- added J-POWRCTL6b-20: 8, TerminalBlock_MetzConnect:TerminalBlock_MetzConnect_360271_1x01_Horizontal_ScrewM3.0_Boxed, F.Cu at (743.9, 116.7)
- added J-POWRCTL6b-21: 8, TerminalBlock_MetzConnect:TerminalBlock_MetzConnect_360271_1x01_Horizontal_ScrewM3.0_Boxed, F.Cu at (760.7, 98.0)
- added J-POWRCTL6b-22: 10, TerminalBlock_MetzConnect:TerminalBlock_MetzConnect_360271_1x01_Horizontal_ScrewM3.0_Boxed, F.Cu at (749.7, 98.0)
- added J-POWRCTL6b-23: , TerminalBlock_MetzConnect:TerminalBlock_MetzConnect_360271_1x01_Horizontal_ScrewM3.0_Boxed, F.Cu at (727.6, 88.7)
- added J-POWRCTL6b-24: , TerminalBlock_MetzConnect:TerminalBlock_MetzConnect_360271_1x01_Horizontal_ScrewM3.0_Boxed, F.Cu at (687.5, 134.9)
- added J-POWRCTL6b-25: 12, TerminalBlock_MetzConnect:TerminalBlock_MetzConnect_360271_1x01_Horizontal_ScrewM3.0_Boxed, F.Cu at (738.6, 88.7)
- added J-POWRCTL6b-26: 11, TerminalBlock_MetzConnect:TerminalBlock_MetzConnect_360271_1x01_Horizontal_ScrewM3.0_Boxed, F.Cu at (698.5, 132.3)
- added J-POWRCTL6b-27: , TerminalBlock_MetzConnect:TerminalBlock_MetzConnect_360271_1x01_Horizontal_ScrewM3.0_Boxed, F.Cu at (676.4, 153.6)
- added J-POWRCTL6b-28: , TerminalBlock_MetzConnect:TerminalBlock_MetzConnect_360271_1x01_Horizontal_ScrewM3.0_Boxed, F.Cu at (721.8, 113.6)
- added J-POWRCTL6b-29: , TerminalBlock_MetzConnect:TerminalBlock_MetzConnect_360271_1x01_Horizontal_ScrewM3.0_Boxed, F.Cu at (738.6, 98.0)
- added J-POWRCTL6b-3: L, TerminalBlock_MetzConnect:TerminalBlock_MetzConnect_360271_1x01_Horizontal_ScrewM3.0_Boxed, F.Cu at (760.7, 88.7)
- added J-POWRCTL6b-30: , TerminalBlock_MetzConnect:TerminalBlock_MetzConnect_360271_1x01_Horizontal_ScrewM3.0_Boxed, F.Cu at (687.5, 153.6)
- added J-POWRCTL6b-31: , TerminalBlock_MetzConnect:TerminalBlock_MetzConnect_360271_1x01_Horizontal_ScrewM3.0_Boxed, F.Cu at (698.5, 141.7)
- added J-POWRCTL6b-32: , TerminalBlock_MetzConnect:TerminalBlock_MetzConnect_360271_1x01_Horizontal_ScrewM3.0_Boxed, F.Cu at (749.7, 88.7)
- added J-POWRCTL6b-33: 5, TerminalBlock_MetzConnect:TerminalBlock_MetzConnect_360271_1x01_Horizontal_ScrewM3.0_Boxed, F.Cu at (709.6, 132.3)
- added J-POWRCTL6b-34: 4, TerminalBlock_MetzConnect:TerminalBlock_MetzConnect_360271_1x01_Horizontal_ScrewM3.0_Boxed, F.Cu at (721.8, 123.0)
- added J-POWRCTL6b-35: 3, TerminalBlock_MetzConnect:TerminalBlock_MetzConnect_360271_1x01_Horizontal_ScrewM3.0_Boxed, F.Cu at (732.8, 107.4)
- added J-POWRCTL6b-36: 2, TerminalBlock_MetzConnect:TerminalBlock_MetzConnect_360271_1x01_Horizontal_ScrewM3.0_Boxed, F.Cu at (676.4, 134.9)
- added J-POWRCTL6b-37: 3, TerminalBlock_MetzConnect:TerminalBlock_MetzConnect_360271_1x01_Horizontal_ScrewM3.0_Boxed, F.Cu at (681.1, 125.5)
- added J-POWRCTL6b-38: 5, TerminalBlock_MetzConnect:TerminalBlock_MetzConnect_360271_1x01_Horizontal_ScrewM3.0_Boxed, F.Cu at (676.4, 144.2)
- added J-POWRCTL6b-39: 4, TerminalBlock_MetzConnect:TerminalBlock_MetzConnect_360271_1x01_Horizontal_ScrewM3.0_Boxed, F.Cu at (710.7, 113.6)
- added J-POWRCTL6b-4: L, TerminalBlock_MetzConnect:TerminalBlock_MetzConnect_360271_1x01_Horizontal_ScrewM3.0_Boxed, F.Cu at (732.8, 116.7)
- added J-POWRCTL6b-40: 3, TerminalBlock_MetzConnect:TerminalBlock_MetzConnect_360271_1x01_Horizontal_ScrewM3.0_Boxed, F.Cu at (727.6, 98.0)
- added J-POWRCTL6b-41: 2, TerminalBlock_MetzConnect:TerminalBlock_MetzConnect_360271_1x01_Horizontal_ScrewM3.0_Boxed, F.Cu at (743.9, 126.1)
- added J-POWRCTL6b-42: 3, TerminalBlock_MetzConnect:TerminalBlock_MetzConnect_360271_1x01_Horizontal_ScrewM3.0_Boxed, F.Cu at (720.6, 141.7)
- added J-POWRCTL6b-5: L, TerminalBlock_MetzConnect:TerminalBlock_MetzConnect_360271_1x01_Horizontal_ScrewM3.0_Boxed, F.Cu at (709.6, 141.7)
- added J-POWRCTL6b-6: 1, TerminalBlock_MetzConnect:TerminalBlock_MetzConnect_360271_1x01_Horizontal_ScrewM3.0_Boxed, F.Cu at (681.1, 116.2)
- added J-POWRCTL6b-7: 1, TerminalBlock_MetzConnect:TerminalBlock_MetzConnect_360271_1x01_Horizontal_ScrewM3.0_Boxed, F.Cu at (699.7, 113.6)
- added J-POWRCTL6b-8: 2, TerminalBlock_MetzConnect:TerminalBlock_MetzConnect_360271_1x01_Horizontal_ScrewM3.0_Boxed, F.Cu at (699.7, 123.0)
- added J-POWRCTL6b-9: 2, TerminalBlock_MetzConnect:TerminalBlock_MetzConnect_360271_1x01_Horizontal_ScrewM3.0_Boxed, F.Cu at (687.5, 144.2)
- added MES-POWRCTL6b-1: 7V, Connector_PinHeader_2.54mm:PinHeader_1x02_P2.54mm_Vertical, F.Cu at (760.9, 139.2)
- added MES-POWRCTL6b-2: 10A, Connector_PinHeader_2.54mm:PinHeader_1x02_P2.54mm_Vertical, F.Cu at (794.6, 86.3)
- added MES-POWRCTL6b-3: 5A, Connector_PinHeader_2.54mm:PinHeader_1x02_P2.54mm_Vertical, F.Cu at (765.6, 139.2)
- added MES-POWRCTL6b-4: 5A, Connector_PinHeader_2.54mm:PinHeader_1x02_P2.54mm_Vertical, F.Cu at (776.5, 127.7)
- added MES-POWRCTL6b-5: 7V, Connector_PinHeader_2.54mm:PinHeader_1x02_P2.54mm_Vertical, F.Cu at (792.2, 111.5)
- added MES-POWRCTL6b-6: 7V, Connector_PinHeader_2.54mm:PinHeader_1x02_P2.54mm_Vertical, F.Cu at (796.3, 103.7)
- added MES-POWRCTL6b-7: 7V, Connector_PinHeader_2.54mm:PinHeader_1x02_P2.54mm_Vertical, F.Cu at (781.1, 120.5)
- added P-POWRCTL6b-1: Conn_WallPlug, Connector_PinHeader_2.54mm:PinHeader_1x02_P2.54mm_Vertical, F.Cu at (753.2, 148.9)
- added PSU-POWRCTL6b-1: PSU-SSEM, Connector_PinHeader_2.54mm:PinHeader_1x09_P2.54mm_Vertical, F.Cu at (715.1, 86.3)
- added PSU-POWRCTL6b-2: PSU-SSEM, Connector_PinHeader_2.54mm:PinHeader_1x09_P2.54mm_Vertical, F.Cu at (710.4, 86.3)
- added PSU-POWRCTL6b-3: PSU-SSEM, Connector_PinHeader_2.54mm:PinHeader_1x09_P2.54mm_Vertical, F.Cu at (705.8, 86.3)
- added PSU-POWRCTL6b-4: PSU-SSEM, Connector_PinHeader_2.54mm:PinHeader_1x09_P2.54mm_Vertical, F.Cu at (701.1, 86.3)
- added PSU-POWRCTL6b-5: PSU-SSEM, Connector_PinHeader_2.54mm:PinHeader_1x09_P2.54mm_Vertical, F.Cu at (696.5, 86.3)
- added PSU-POWRCTL6b-6: PSU-SSEM, Connector_PinHeader_2.54mm:PinHeader_1x09_P2.54mm_Vertical, F.Cu at (691.8, 86.3)
- added R-POWRCTL6b-1: 2R 3W, Resistor_THT:R_Axial_DIN0516_L15.5mm_D5.0mm_P5.08mm_Vertical, F.Cu at (763.7, 106.0)
- added R-POWRCTL6b-2: 2R 3W, Resistor_THT:R_Axial_DIN0516_L15.5mm_D5.0mm_P5.08mm_Vertical, F.Cu at (718.4, 149.6)
- added R-POWRCTL6b-3: 2R 3W, Resistor_THT:R_Axial_DIN0516_L15.5mm_D5.0mm_P5.08mm_Vertical, F.Cu at (780.6, 87.3)
- added RV-POWRCTL6b-1: 17R, Connector_PinHeader_2.54mm:PinHeader_1x03_P2.54mm_Vertical, F.Cu at (762.8, 111.6)
- added RV-POWRCTL6b-2: 17R, Connector_PinHeader_2.54mm:PinHeader_1x03_P2.54mm_Vertical, F.Cu at (751.7, 123.7)
- added RV-POWRCTL6b-3: 17R, Connector_PinHeader_2.54mm:PinHeader_1x03_P2.54mm_Vertical, F.Cu at (739.5, 133.1)
- added SW-POWRCTL6b-1: SW_SPST, Connector_PinHeader_2.54mm:PinHeader_1x04_P2.54mm_Vertical, F.Cu at (673.2, 113.8)
- added SW-POWRCTL6b-2: SW_Push, Connector_PinHeader_2.54mm:PinHeader_1x02_P2.54mm_Vertical, F.Cu at (796.8, 110.9)
- added SW-POWRCTL6b-3: SW_Push_Open, Connector_PinHeader_2.54mm:PinHeader_1x02_P2.54mm_Vertical, F.Cu at (757.9, 148.9)
- added SW-POWRCTL6b-4: SW_SPDT, Connector_PinHeader_2.54mm:PinHeader_1x03_P2.54mm_Vertical, F.Cu at (733.1, 142.4)
- added SW-POWRCTL6b-5: SW_SPDT, Connector_PinHeader_2.54mm:PinHeader_1x03_P2.54mm_Vertical, F.Cu at (779.6, 92.9)
- added SW-POWRCTL6b-6: SW_SPDT, Connector_PinHeader_2.54mm:PinHeader_1x03_P2.54mm_Vertical, F.Cu at (790.0, 86.3)
- added T-POWRCTL6b-1: Transformer_1P_2S, Connector_PinHeader_2.54mm:PinHeader_1x06_P2.54mm_Vertical, F.Cu at (691.8, 111.3)
- added T-POWRCTL6b-2: Transformer_1P_2S, Connector_PinHeader_2.54mm:PinHeader_1x06_P2.54mm_Vertical, F.Cu at (668.6, 141.3)
- added TR-POWRCTL6b-1: VARIAC, Connector_PinHeader_2.54mm:PinHeader_1x03_P2.54mm_Vertical, F.Cu at (728.5, 142.4)
- added V-POWRCTL6b-1: CV71, Connector_PinHeader_2.54mm:PinHeader_1x02_P2.54mm_Vertical, F.Cu at (781.1, 127.7)
- added V-POWRCTL6b-2: CV71, Connector_PinHeader_2.54mm:PinHeader_1x02_P2.54mm_Vertical, F.Cu at (770.2, 134.9)
- added V-POWRCTL6b-3: CV71, Connector_PinHeader_2.54mm:PinHeader_1x02_P2.54mm_Vertical, F.Cu at (785.8, 118.7)
- added V-POWRCTL6b-4: CV71, Connector_PinHeader_2.54mm:PinHeader_1x02_P2.54mm_Vertical, F.Cu at (719.7, 103.7)
- J-KVPSU1-1, J-KVPSU1-10, J-KVPSU1-2, J-KVPSU1-4, J-KVPSU1-5, J-KVPSU1-6, J-KVPSU1-7, J-KVPSU1-9: footprint SamacSys_Parts_l:242431 -> TerminalBlock_MetzConnect:TerminalBlock_MetzConnect_360271_1x01_Horizontal_ScrewM3.0_Boxed
- V-KVPSU2-4: footprint Valve:Valve_Octal -> Connector_PinHeader_2.54mm:PinHeader_1x02_P2.54mm_Vertical
- moved J-KEYSW2-5 719.6 mm to (-3.56, 343.0)
- moved SW8 706.1 mm to (51.8, 356.0)
- moved R-KEYSW2-1 703.0 mm to (11.7, 381.1)
- moved J-KEYSW2-6 698.2 mm to (-12.9, 375.6)
- moved SW10 697.3 mm to (47.2, 356.0)
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Connections:
- D-CRTCCT3-1 pad 2: /CRTCCT3/S.EHT(800-1400V) -> (no net)
- D-CRTCCT5-1 pad 2: (no net) -> /CRTCCT5/S.EHT(800-1400V)

Commit message: Add Prepulse PSEPCTL RMONDRS.
Signed-off-by: John Bradley <flypie@rocketmail.com>
Parts:
- added C-PREPULSE--A-1: 0.5, Capacitor_THT:C_Disc_D7.5mm_W5.0mm_P5.00mm, F.Cu at (239.0, 193.9)
- added C-PREPULSE-1: 220p, Capacitor_THT:C_Disc_D7.5mm_W5.0mm_P5.00mm, F.Cu at (224.1, 207.0)
- added C-PREPULSE-10: 0.1u, Capacitor_THT:C_Disc_D7.5mm_W5.0mm_P5.00mm, F.Cu at (189.0, 249.6)
- added C-PREPULSE-11: 100pf, Capacitor_THT:C_Disc_D7.5mm_W5.0mm_P5.00mm, F.Cu at (208.9, 227.2)
- added C-PREPULSE-12: 100pf, Capacitor_THT:C_Disc_D7.5mm_W5.0mm_P5.00mm, F.Cu at (202.7, 233.7)
- added C-PREPULSE-13: 100pf, Capacitor_THT:C_Disc_D7.5mm_W5.0mm_P5.00mm, F.Cu at (249.3, 187.3)
- added C-PREPULSE-14: 100pf, Capacitor_THT:C_Disc_D7.5mm_W5.0mm_P5.00mm, F.Cu at (193.7, 240.3)
- added C-PREPULSE-15: 220pf, Capacitor_THT:C_Disc_D7.5mm_W5.0mm_P5.00mm, F.Cu at (234.4, 200.4)
- added C-PREPULSE-2: 2800pf, Capacitor_THT:C_Disc_D7.5mm_W5.0mm_P5.00mm, F.Cu at (210.2, 220.6)
- added C-PREPULSE-3: 0.5, Capacitor_THT:C_Disc_D7.5mm_W5.0mm_P5.00mm, F.Cu at (193.7, 233.7)
- added C-PREPULSE-4: 100p, Capacitor_THT:C_Disc_D7.5mm_W5.0mm_P5.00mm, F.Cu at (199.9, 227.2)
- added C-PREPULSE-5: 0.5, Capacitor_THT:C_Disc_D7.5mm_W5.0mm_P5.00mm, F.Cu at (180.0, 250.3)
- added C-PREPULSE-6: 0.5, Capacitor_THT:C_Disc_D7.5mm_W5.0mm_P5.00mm, F.Cu at (226.9, 213.5)
- added C-PREPULSE-7: 0.1u, Capacitor_THT:C_Disc_D7.5mm_W5.0mm_P5.00mm, F.Cu at (233.1, 207.0)
- added C-PREPULSE-8: 47p, Capacitor_THT:C_Disc_D7.5mm_W5.0mm_P5.00mm, F.Cu at (219.3, 220.6)
- added C-PREPULSE-9: 0.1, Capacitor_THT:C_Disc_D7.5mm_W5.0mm_P5.00mm, F.Cu at (217.9, 214.1)
- added C-PSEPCTL--A-1: 0.5, Capacitor_THT:C_Disc_D7.5mm_W5.0mm_P5.00mm, F.Cu at (543.9, 413.7)
- added C-PSEPCTL-1: 0.01uf, Capacitor_THT:C_Disc_D7.5mm_W5.0mm_P5.00mm, F.Cu at (541.2, 420.2)
- added C-PSEPCTL-2: 0.1uf, Capacitor_THT:C_Disc_D7.5mm_W5.0mm_P5.00mm, F.Cu at (554.3, 403.7)
- added C-PSEPCTL-3: 0.5, Capacitor_THT:C_Disc_D7.5mm_W5.0mm_P5.00mm, F.Cu at (566.0, 394.0)
- added C-PSEPCTL-4: 0.01uf, Capacitor_THT:C_Disc_D7.5mm_W5.0mm_P5.00mm, F.Cu at (508.3, 445.7)
- added C-PSEPCTL-5: 0.5, Capacitor_THT:C_Disc_D7.5mm_W5.0mm_P5.00mm, F.Cu at (518.7, 443.8)
- added C-PSEPCTL-6: 0.5, Capacitor_THT:C_Disc_D7.5mm_W5.0mm_P5.00mm, F.Cu at (527.7, 436.4)
- added C-PSEPCTL-7: 0.25uf, Capacitor_THT:C_Disc_D7.5mm_W5.0mm_P5.00mm, F.Cu at (554.3, 410.2)
- added C-PSEPCTL-8: 0.25uf, Capacitor_THT:C_Disc_D7.5mm_W5.0mm_P5.00mm, F.Cu at (530.9, 429.8)
- added C-PSEPCTL-9: 0.1uf, Capacitor_THT:C_Disc_D7.5mm_W5.0mm_P5.00mm, F.Cu at (518.7, 437.3)
- added C-RMONDRS--A-1: 0.5, Capacitor_THT:C_Disc_D7.5mm_W5.0mm_P5.00mm, F.Cu at (182.5, 457.1)
- added C-RMONDRS-1: 0.1uf, Capacitor_THT:C_Disc_D7.5mm_W5.0mm_P5.00mm, F.Cu at (220.0, 418.1)
- added C-RMONDRS-10: 0.1uf, Capacitor_THT:C_Disc_D7.5mm_W5.0mm_P5.00mm, F.Cu at (235.3, 405.9)
- added C-RMONDRS-11: 0.5uf, Capacitor_THT:C_Disc_D7.5mm_W5.0mm_P5.00mm, F.Cu at (192.9, 445.7)
- added C-RMONDRS-2: 0.1uf, Capacitor_THT:C_Disc_D7.5mm_W5.0mm_P5.00mm, F.Cu at (220.0, 424.6)
- added C-RMONDRS-3: 0.5, Capacitor_THT:C_Disc_D7.5mm_W5.0mm_P5.00mm, F.Cu at (209.3, 439.2)
- added C-RMONDRS-4: 0.1uf, Capacitor_THT:C_Disc_D7.5mm_W5.0mm_P5.00mm, F.Cu at (229.1, 412.4)
- added C-RMONDRS-5: 0.5, Capacitor_THT:C_Disc_D7.5mm_W5.0mm_P5.00mm, F.Cu at (235.3, 399.3)
- added C-RMONDRS-6: 0.5, Capacitor_THT:C_Disc_D7.5mm_W5.0mm_P5.00mm, F.Cu at (192.9, 452.3)
- added C-RMONDRS-7: 0.5uf, Capacitor_THT:C_Disc_D7.5mm_W5.0mm_P5.00mm, F.Cu at (182.5, 463.6)
- added C-RMONDRS-8: 0.1uf, Capacitor_THT:C_Disc_D7.5mm_W5.0mm_P5.00mm, F.Cu at (244.3, 399.3)
- added C-RMONDRS-9: 0.5uf, Capacitor_THT:C_Disc_D7.5mm_W5.0mm_P5.00mm, F.Cu at (209.3, 432.6)
- added D-PREPULSE-1: EA50, NewValves:Valve_B3G, F.Cu at (207.0, 178.0)
- added D-PREPULSE-10: EA50, NewValves:Valve_B3G, F.Cu at (221.9, 170.9)
- added D-PREPULSE-11: EA50, NewValves:Valve_B3G, F.Cu at (208.0, 191.1)
- added D-PREPULSE-12: EA50, NewValves:Valve_B3G, F.Cu at (243.6, 157.8)
- added D-PREPULSE-13: EA50, NewValves:Valve_B3G, F.Cu at (178.2, 200.4)
- added D-PREPULSE-14: EA50, NewValves:Valve_B3G, F.Cu at (179.2, 226.7)
- added D-PREPULSE-15: EA50, NewValves:Valve_B3G, F.Cu at (149.4, 229.2)
- added D-PREPULSE-16: EA50, NewValves:Valve_B3G, F.Cu at (213.8, 157.8)
- added D-PREPULSE-17: EA50, NewValves:Valve_B3G, F.Cu at (161.6, 214.3)
- added D-PREPULSE-18: EA50, NewValves:Valve_B3G, F.Cu at (134.5, 229.2)
- added D-PREPULSE-19: EA50, NewValves:Valve_B3G, F.Cu at (163.3, 200.4)
- added D-PREPULSE-2: EA50, NewValves:Valve_B3G, F.Cu at (228.7, 157.8)
- added D-PREPULSE-20: EA50, NewValves:Valve_B3G, F.Cu at (192.1, 178.0)
- added D-PREPULSE-3: EA50, NewValves:Valve_B3G, F.Cu at (132.9, 243.0)
- added D-PREPULSE-4: EA50, NewValves:Valve_B3G, F.Cu at (147.8, 242.3)
- added D-PREPULSE-5: EA50, NewValves:Valve_B3G, F.Cu at (176.5, 213.5)
- added D-PREPULSE-6: EA50, NewValves:Valve_B3G, F.Cu at (164.3, 227.4)
- added D-PREPULSE-7: EA50, NewValves:Valve_B3G, F.Cu at (193.1, 191.1)
- added D-PREPULSE-8: EA50, NewValves:Valve_B3G, F.Cu at (162.6, 242.3)
- added D-PREPULSE-9: EA50, NewValves:Valve_B3G, F.Cu at (193.1, 204.3)
- added D-PSEPCTL-1: EA50, NewValves:Valve_B3G, F.Cu at (545.2, 371.1)
- added D-PSEPCTL-2: EA50, NewValves:Valve_B3G, F.Cu at (545.2, 384.2)
- added D-PSEPCTL-3: EA50, NewValves:Valve_B3G, F.Cu at (487.7, 442.4)
- added D-RMONDRS-1: D, Diode_THT:D_5W_P5.08mm_Vertical_KathodeUp, F.Cu at (189.9, 439.7)
- added D-RMONDRS-2: D, Diode_THT:D_5W_P5.08mm_Vertical_KathodeUp, F.Cu at (205.2, 426.6)
- added D-RMONDRS-3: D, Diode_THT:D_5W_P5.08mm_Vertical_KathodeUp, F.Cu at (215.5, 412.1)
- added J-PREPULSE-1: C0, SamacSys_Parts_l:242431, F.Cu at (164.2, 171.7)
- added J-PREPULSE-10: HA, SamacSys_Parts_l:242431, F.Cu at (133.8, 215.4)
- added J-PREPULSE-11: Completion Signal (Prepulse), SamacSys_Parts_l:242431, F.Cu at (162.5, 186.7)
- added J-PREPULSE-2: HIGH Voltage., Connector_TE-Connectivity:TE_MATE-N-LOK_1-770970-x_2x04_P4.14mm_Horizontal, F.Cu at (187.9, 155.1)
- added J-PREPULSE-3: Completion Signal (Prepulse), SamacSys_Parts_l:242431, F.Cu at (135.4, 186.7)
- added J-PREPULSE-4: P0.CF, SamacSys_Parts_l:242431, F.Cu at (106.7, 215.4)
- added J-PREPULSE-5: P1.CF, SamacSys_Parts_l:242431, F.Cu at (77.9, 244.2)
- added J-PREPULSE-6: Plus1, SamacSys_Parts_l:242431, F.Cu at (164.2, 157.9)
- added J-PREPULSE-7: Plus2, SamacSys_Parts_l:242431, F.Cu at (105.0, 244.2)
- added J-PREPULSE-8: Plus1or2, SamacSys_Parts_l:242431, F.Cu at (135.4, 200.5)
- added J-PREPULSE-9: C0, SamacSys_Parts_l:242431, F.Cu at (106.7, 229.3)
- added J-PSEPCTL-1: DASH, SamacSys_Parts_l:242431, F.Cu at (488.6, 413.7)
- added J-PSEPCTL-2: HIGH Voltage., Connector_TE-Connectivity:TE_MATE-N-LOK_1-770970-x_2x04_P4.14mm_Horizontal, F.Cu at (512.2, 397.1)
- added J-PSEPCTL-3: POS.DASH, SamacSys_Parts_l:242431, F.Cu at (517.3, 385.0)
- added J-PSEPCTL-4: P0, SamacSys_Parts_l:242431, F.Cu at (486.9, 428.7)
- added J-PSEPCTL-5: P1, SamacSys_Parts_l:242431, F.Cu at (459.8, 442.5)
- added J-PSEPCTL-6: P0.CF, SamacSys_Parts_l:242431, F.Cu at (517.3, 371.1)
- added J-PSEPCTL-7: P1.CF, SamacSys_Parts_l:242431, F.Cu at (488.6, 399.9)
- added J-PSEPCTL-8: +20V, SamacSys_Parts_l:242431, F.Cu at (459.8, 428.7)
- added J-RMONDRS-1: S.Read, SamacSys_Parts_l:242431, F.Cu at (105.0, 462.3)
- added J-RMONDRS-10: M.X2, SamacSys_Parts_l:242431, F.Cu at (135.4, 447.3)
- added J-RMONDRS-11: Y2, SamacSys_Parts_l:242431, F.Cu at (164.2, 417.3)
- added J-RMONDRS-12: Y1, SamacSys_Parts_l:242431, F.Cu at (191.3, 389.8)
- added J-RMONDRS-13: R.X2, SamacSys_Parts_l:242431, F.Cu at (162.5, 433.5)
- added J-RMONDRS-14: Conn_02x06_Odd_Even, Connector_PinHeader_2.54mm:PinHeader_2x06_P2.54mm_Vertical, F.Cu at (187.8, 413.1)
- added J-RMONDRS-15: Y2, SamacSys_Parts_l:242431, F.Cu at (191.3, 403.6)
- added J-RMONDRS-2: HIGH Voltage., Connector_TE-Connectivity:TE_MATE-N-LOK_1-770970-x_2x04_P4.14mm_Horizontal, F.Cu at (228.4, 373.2)
- added J-RMONDRS-3: Diff.Dot, SamacSys_Parts_l:242431, F.Cu at (77.9, 462.3)
- added J-RMONDRS-4: Ha, SamacSys_Parts_l:242431, F.Cu at (177.6, 375.9)
- added J-RMONDRS-5: S.GRID, SamacSys_Parts_l:242431, F.Cu at (164.2, 403.4)
- added J-RMONDRS-6: R.X1, SamacSys_Parts_l:242431, F.Cu at (135.4, 433.5)
- added J-RMONDRS-7: R.Grid, SamacSys_Parts_l:242431, F.Cu at (204.7, 375.9)
- added J-RMONDRS-8: M.X1, SamacSys_Parts_l:242431, F.Cu at (132.1, 462.3)
- added J-RMONDRS-9: Y2, SamacSys_Parts_l:242431, F.Cu at (159.2, 461.1)
- added R-PREPULSE-1: 51K, Resistor_THT:R_Axial_DIN0516_L15.5mm_D5.0mm_P5.08mm_Vertical, F.Cu at (174.2, 237.2)
- added R-PREPULSE-10: 220uf, Resistor_THT:R_Axial_DIN0516_L15.5mm_D5.0mm_P5.08mm_Vertical, F.Cu at (233.5, 174.2)
- added R-PREPULSE-11: 470, Resistor_THT:R_Axial_DIN0516_L15.5mm_D5.0mm_P5.08mm_Vertical, F.Cu at (228.9, 180.8)
- added R-PREPULSE-12: 220K, Resistor_THT:R_Axial_DIN0516_L15.5mm_D5.0mm_P5.08mm_Vertical, F.Cu at (243.8, 167.7)
- added R-PREPULSE-13: 3K9 6W, Resistor_THT:R_Axial_DIN0516_L15.5mm_D5.0mm_P5.08mm_Vertical, F.Cu at (233.5, 167.7)
- added R-PREPULSE-14: 10M, Resistor_THT:R_Axial_DIN0516_L15.5mm_D5.0mm_P5.08mm_Vertical, F.Cu at (219.6, 193.9)
- added R-PREPULSE-15: 47K, Resistor_THT:R_Axial_DIN0516_L15.5mm_D5.0mm_P5.08mm_Vertical, F.Cu at (190.8, 220.6)
- added R-PREPULSE-16: 470, Resistor_THT:R_Axial_DIN0516_L15.5mm_D5.0mm_P5.08mm_Vertical, F.Cu at (85.7, 254.7)
- added R-PREPULSE-17: 750, Resistor_THT:R_Axial_DIN0516_L15.5mm_D5.0mm_P5.08mm_Vertical, F.Cu at (129.6, 252.9)
- added R-PREPULSE-18: 15K 2W, Resistor_THT:R_Axial_DIN0516_L15.5mm_D5.0mm_P5.08mm_Vertical, F.Cu at (116.7, 254.7)
- added R-PREPULSE-19: 10K 3W, Resistor_THT:R_Axial_DIN0516_L15.5mm_D5.0mm_P5.08mm_Vertical, F.Cu at (75.4, 254.7)
- added R-PREPULSE-2: 470, Resistor_THT:R_Axial_DIN0516_L15.5mm_D5.0mm_P5.08mm_Vertical, F.Cu at (198.5, 214.1)
- added R-PREPULSE-20: 1M, Resistor_THT:R_Axial_DIN0516_L15.5mm_D5.0mm_P5.08mm_Vertical, F.Cu at (150.2, 252.1)
- added R-PREPULSE-21: 470, Resistor_THT:R_Axial_DIN0516_L15.5mm_D5.0mm_P5.08mm_Vertical, F.Cu at (204.7, 201.0)
- added R-PREPULSE-22: 47K, Resistor_THT:R_Axial_DIN0516_L15.5mm_D5.0mm_P5.08mm_Vertical, F.Cu at (229.9, 193.9)
- added R-PREPULSE-23: 470K, Resistor_THT:R_Axial_DIN0516_L15.5mm_D5.0mm_P5.08mm_Vertical, F.Cu at (188.1, 214.1)
- added R-PREPULSE-24: 470, Resistor_THT:R_Axial_DIN0516_L15.5mm_D5.0mm_P5.08mm_Vertical, F.Cu at (249.6, 180.8)
- added R-PREPULSE-25: 39K 1W, Resistor_THT:R_Axial_DIN0516_L15.5mm_D5.0mm_P5.08mm_Vertical, F.Cu at (184.6, 243.0)
- added R-PREPULSE-26: 220K, Resistor_THT:R_Axial_DIN0516_L15.5mm_D5.0mm_P5.08mm_Vertical, F.Cu at (254.1, 174.2)
- added R-PREPULSE-27: 470, Resistor_THT:R_Axial_DIN0516_L15.5mm_D5.0mm_P5.08mm_Vertical, F.Cu at (240.2, 187.3)
- added R-PREPULSE-28: 330K, Resistor_THT:R_Axial_DIN0516_L15.5mm_D5.0mm_P5.08mm_Vertical, F.Cu at (225.3, 200.4)
- added R-PREPULSE-29: 470K, Resistor_THT:R_Axial_DIN0516_L15.5mm_D5.0mm_P5.08mm_Vertical, F.Cu at (106.4, 254.7)
- added R-PREPULSE-3: 1M, Resistor_THT:R_Axial_DIN0516_L15.5mm_D5.0mm_P5.08mm_Vertical, F.Cu at (215.0, 201.0)
- added R-PREPULSE-30: 10K 3W, Resistor_THT:R_Axial_DIN0516_L15.5mm_D5.0mm_P5.08mm_Vertical, F.Cu at (160.6, 252.1)
- added R-PREPULSE-31: 47K 2W, Resistor_THT:R_Axial_DIN0516_L15.5mm_D5.0mm_P5.08mm_Vertical, F.Cu at (204.7, 207.5)
- added R-PREPULSE-32: 68K 3W, Resistor_THT:R_Axial_DIN0516_L15.5mm_D5.0mm_P5.08mm_Vertical, F.Cu at (201.1, 220.6)
- added R-PREPULSE-33: 470, Resistor_THT:R_Axial_DIN0516_L15.5mm_D5.0mm_P5.08mm_Vertical, F.Cu at (215.0, 207.5)
- added R-PREPULSE-34: 1M, Resistor_THT:R_Axial_DIN0516_L15.5mm_D5.0mm_P5.08mm_Vertical, F.Cu at (170.9, 252.1)
- added R-PREPULSE-35: 12K 2W, Resistor_THT:R_Axial_DIN0516_L15.5mm_D5.0mm_P5.08mm_Vertical, F.Cu at (208.8, 214.1)
- added R-PREPULSE-36: 820K, Resistor_THT:R_Axial_DIN0516_L15.5mm_D5.0mm_P5.08mm_Vertical, F.Cu at (243.8, 174.2)
- added R-PREPULSE-37: 470, Resistor_THT:R_Axial_DIN0516_L15.5mm_D5.0mm_P5.08mm_Vertical, F.Cu at (254.1, 167.7)
- added R-PREPULSE-38: 3.3k6W, Resistor_THT:R_Axial_DIN0516_L15.5mm_D5.0mm_P5.08mm_Vertical, F.Cu at (174.2, 243.8)
- added R-PREPULSE-39: 470K, Resistor_THT:R_Axial_DIN0516_L15.5mm_D5.0mm_P5.08mm_Vertical, F.Cu at (190.8, 227.2)
- added R-PREPULSE-4: 100K, Resistor_THT:R_Axial_DIN0516_L15.5mm_D5.0mm_P5.08mm_Vertical, F.Cu at (229.9, 187.3)
- added R-PREPULSE-40: 22K, Resistor_THT:R_Axial_DIN0516_L15.5mm_D5.0mm_P5.08mm_Vertical, F.Cu at (239.2, 180.8)
- added R-PREPULSE-5: 68K, Resistor_THT:R_Axial_DIN0516_L15.5mm_D5.0mm_P5.08mm_Vertical, F.Cu at (184.6, 236.5)
- added R-PREPULSE-6: 100K, Resistor_THT:R_Axial_DIN0516_L15.5mm_D5.0mm_P5.08mm_Vertical, F.Cu at (96.0, 254.7)
- added R-PREPULSE-7: 39K, Resistor_THT:R_Axial_DIN0516_L15.5mm_D5.0mm_P5.08mm_Vertical, F.Cu at (139.9, 252.9)
- added R-PREPULSE-8: 47K, Resistor_THT:R_Axial_DIN0516_L15.5mm_D5.0mm_P5.08mm_Vertical, F.Cu at (218.6, 180.8)
- added R-PREPULSE-9: 51K, Resistor_THT:R_Axial_DIN0516_L15.5mm_D5.0mm_P5.08mm_Vertical, F.Cu at (219.6, 187.3)
- added R-PSEPCTL-1: 6K8, Resistor_THT:R_Axial_DIN0516_L15.5mm_D5.0mm_P5.08mm_Vertical, F.Cu at (556.8, 387.4)
- added R-PSEPCTL-10: 100k, Resistor_THT:R_Axial_DIN0516_L15.5mm_D5.0mm_P5.08mm_Vertical, F.Cu at (567.1, 380.9)
- added R-PSEPCTL-11: 47, Resistor_THT:R_Axial_DIN0516_L15.5mm_D5.0mm_P5.08mm_Vertical, F.Cu at (521.8, 429.8)
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Connections:
- D-CRTCCT3-1 pad 2: (no net) -> /CRTCCT3/S.EHT(800-1400V)
- U-CRTPCIF2-5 pad 8: /CRTPCIF2/Bk1 -> (no net)

Commit message: Add scfollws.sch
Signed-off-by: John Bradley <flypie@rocketmail.com>
Parts:
- removed the C-ACTN_WF-3 at (983.0, 35.7)
- removed the C-CMOSCRT1-4 at (654.4, 522.5)
- removed the C-CRTAMP3-20 at (713.4, 217.2)
- removed the C-CRTAMP3-35 at (769.3, 181.2)
- removed the C-CRTAMP3-5 at (782.3, 141.9)
- removed the C-CRTAMP4-17 at (343.2, 436.6)
- removed the C-CRTAMP4-2 at (352.2, 436.6)
- removed the C-CRTAMP4-32 at (388.7, 400.5)
- removed the C-CRTAMP4-47 at (399.1, 413.6)
- removed the C-CRTCCT4-5 at (687.0, 386.2)
- removed the C-CRTPCIF2-6 at (352.7, 536.4)
- removed the C-CTRLGATE-9 at (797.7, 83.0)
- removed the C-FSTAT15-10 at (403.9, 221.5)
- removed the C-IGYSH3-8 at (174.2, 361.5)
- removed the C-PREPULSE-7 at (233.1, 207.0)
- removed the C-PSEPCTL-6 at (527.7, 436.4)
- removed the C-RMONDRS-5 at (235.3, 399.3)
- removed the D-ADDER1-15 at (193.1, 100.9)
- removed the D-ADDER1-16A1 at (234.1, 46.3)
- removed the D-ADDER1-8 at (234.1, 59.4)
- removed the D-CMOSCRT2-16 at (101.1, 553.3)
- removed the D-CMOSCRT2-6 at (194.9, 479.6)
- removed the D-CRTCCT4-1 at (709.6, 338.8)
- removed the D-CRTPCIF2-7 at (329.7, 544.7)
- removed the D-CTRLGATE-1 at (787.3, 73.9)
- removed the D2 at (590.5, 544.0)
- removed J-PREPULSE-2: HIGH Voltage., Connector_TE-Connectivity:TE_MATE-N-LOK_1-770970-x_2x04_P4.14mm_Horizontal
- added C-SCFOLLWS--A-1: 0.5, Capacitor_THT:C_Disc_D7.5mm_W5.0mm_P5.00mm, F.Cu at (-41.5, -90.9)
- added C-SCFOLLWS-2: 0.1u, Capacitor_THT:C_Disc_D7.5mm_W5.0mm_P5.00mm, F.Cu at (12.3, -147.3)
- added C-SCFOLLWS-3: 0.5, Capacitor_THT:C_Disc_D7.5mm_W5.0mm_P5.00mm, F.Cu at (-11.3, -125.5)
- added C-SCFOLLWS-5: 0.5, Capacitor_THT:C_Disc_D7.5mm_W5.0mm_P5.00mm, F.Cu at (-26.2, -110.5)
- added C-SCFOLLWS-6: 0.5, Capacitor_THT:C_Disc_D7.5mm_W5.0mm_P5.00mm, F.Cu at (-36.5, -104.0)
- added C-SCFOLLWS-7: 0.1u, Capacitor_THT:C_Disc_D7.5mm_W5.0mm_P5.00mm, F.Cu at (12.3, -153.8)
- added D-SCFOLLWS-1: EA50, NewValves:Valve_B3G, F.Cu at (-42.3, -120.3)
- added D-SCFOLLWS-2: EA50, NewValves:Valve_B3G, F.Cu at (13.6, -176.8)
- added J-SCFOLLWS-1: XBO, SamacSys_Parts_l:242431, F.Cu at (-70.2, -105.6)
- added J-SCFOLLWS-10: XBO.CF, SamacSys_Parts_l:242431, F.Cu at (-156.5, -90.4)
- added J-SCFOLLWS-11: Dot.CF, SamacSys_Parts_l:242431, F.Cu at (-102.3, -90.4)
- added J-SCFOLLWS-12: Var.Dash, SamacSys_Parts_l:242431, F.Cu at (-21.3, -149.0)
- added J-SCFOLLWS-13: XBO.CF, SamacSys_Parts_l:242431, F.Cu at (-41.4, -176.7)
- added J-SCFOLLWS-14: Var.Dash.CF, SamacSys_Parts_l:242431, F.Cu at (-129.4, -90.4)
- added J-SCFOLLWS-15: HIGH Voltage., Connector_TE-Connectivity:TE_MATE-N-LOK_1-770972-x_2x06_P4.14mm_Horizontal, F.Cu at (-325.2, -121.9)
- added J-SCFOLLWS-2: HIGH Voltage., Connector_TE-Connectivity:TE_MATE-N-LOK_1-770972-x_2x06_P4.14mm_Horizontal, F.Cu at (-73.6, -150.7)
- added J-SCFOLLWS-3: Dot.Buff, SamacSys_Parts_l:242431, F.Cu at (-75.2, -90.4)
- added J-SCFOLLWS-4: XBO.CF, SamacSys_Parts_l:242431, F.Cu at (-14.3, -162.9)
- added J-SCFOLLWS-5: Strobe, SamacSys_Parts_l:242431, F.Cu at (-48.4, -134.1)
- added J-SCFOLLWS-6: Dot, SamacSys_Parts_l:242431, F.Cu at (-70.2, -119.5)
- added J-SCFOLLWS-7: Strobe.CF, SamacSys_Parts_l:242431, F.Cu at (-48.4, -147.9)
- added J-SCFOLLWS-8: Diff Dot, SamacSys_Parts_l:242431, F.Cu at (-41.4, -162.9)
- added J-SCFOLLWS-9: Dot, SamacSys_Parts_l:242431, F.Cu at (-14.3, -176.7)
- added R-FSTAT14-5: 560K, Resistor_THT:R_Axial_DIN0516_L15.5mm_D5.0mm_P5.08mm_Vertical, F.Cu at (174.7, -249.9)
- added R-IGYSH3-10: 330K, Resistor_THT:R_Axial_DIN0516_L15.5mm_D5.0mm_P5.08mm_Vertical, F.Cu at (-199.6, -49.9)
- added R-KVPSU1-6: 2R 3W, Resistor_THT:R_Axial_DIN0516_L15.5mm_D5.0mm_P5.08mm_Vertical, F.Cu at (206.3, 200.2)
- added R-KVPSU2-3: 800K, Resistor_THT:R_Axial_DIN0516_L15.5mm_D5.0mm_P5.08mm_Vertical, F.Cu at (288.3, 204.7)
- added R-L-STAT-18: 180K, Resistor_THT:R_Axial_DIN0516_L15.5mm_D5.0mm_P5.08mm_Vertical, F.Cu at (412.5, -298.9)
- added R-MONICCT-4: 470K, Resistor_THT:R_Axial_DIN0516_L15.5mm_D5.0mm_P5.08mm_Vertical, F.Cu at (394.1, -135.0)
- added R-MONSW-15: 330K, Resistor_THT:R_Axial_DIN0516_L15.5mm_D5.0mm_P5.08mm_Vertical, F.Cu at (36.8, -285.8)
- added R-PREPULSE-11: 470, Resistor_THT:R_Axial_DIN0516_L15.5mm_D5.0mm_P5.08mm_Vertical, F.Cu at (-174.3, -160.4)
- added R-PREPULSE-30: 10K 3W, Resistor_THT:R_Axial_DIN0516_L15.5mm_D5.0mm_P5.08mm_Vertical, F.Cu at (-245.7, -104.7)
- added R-PSEPCTL-9: 1M, Resistor_THT:R_Axial_DIN0516_L15.5mm_D5.0mm_P5.08mm_Vertical, F.Cu at (70.8, 106.3)
- added R-RMONDRS-22: 22K 3W, Resistor_THT:R_Axial_DIN0516_L15.5mm_D5.0mm_P5.08mm_Vertical, F.Cu at (-41.1, -14.2)
- added R-RMONDRS-3: 1M, Resistor_THT:R_Axial_DIN0516_L15.5mm_D5.0mm_P5.08mm_Vertical, F.Cu at (2.89, -63.0)
- added R-SCFOLLWS-1: 10K 6W, Resistor_THT:R_Axial_DIN0516_L15.5mm_D5.0mm_P5.08mm_Vertical, F.Cu at (-30.7, -123.6)
- added R-SCFOLLWS-10: 8K2, Resistor_THT:R_Axial_DIN0516_L15.5mm_D5.0mm_P5.08mm_Vertical, F.Cu at (-30.7, -117.1)
- added R-SCFOLLWS-11: 470, Resistor_THT:R_Axial_DIN0516_L15.5mm_D5.0mm_P5.08mm_Vertical, F.Cu at (-40.3, -97.4)
- added R-SCFOLLWS-12: 470, Resistor_THT:R_Axial_DIN0516_L15.5mm_D5.0mm_P5.08mm_Vertical, F.Cu at (-3.21, -138.6)
- added R-SCFOLLWS-13: 10K 6W, Resistor_THT:R_Axial_DIN0516_L15.5mm_D5.0mm_P5.08mm_Vertical, F.Cu at (-20.4, -118.9)
- added R-SCFOLLWS-14: 7K5 6W, Resistor_THT:R_Axial_DIN0516_L15.5mm_D5.0mm_P5.08mm_Vertical, F.Cu at (10.3, -160.4)
- added R-SCFOLLWS-15: 390K, Resistor_THT:R_Axial_DIN0516_L15.5mm_D5.0mm_P5.08mm_Vertical, F.Cu at (-13.5, -132.0)
- added R-SCFOLLWS-16: 470, Resistor_THT:R_Axial_DIN0516_L15.5mm_D5.0mm_P5.08mm_Vertical, F.Cu at (-23.9, -132.0)
- added R-SCFOLLWS-17: 9K 6W, Resistor_THT:R_Axial_DIN0516_L15.5mm_D5.0mm_P5.08mm_Vertical, F.Cu at (-20.4, -125.5)
- added R-SCFOLLWS-18: 470, Resistor_THT:R_Axial_DIN0516_L15.5mm_D5.0mm_P5.08mm_Vertical, F.Cu at (-13.5, -138.6)
- added R-SCFOLLWS-19: 7K5 6W, Resistor_THT:R_Axial_DIN0516_L15.5mm_D5.0mm_P5.08mm_Vertical, F.Cu at (-50.6, -95.2)
- added R-SCFOLLWS-2: 470, Resistor_THT:R_Axial_DIN0516_L15.5mm_D5.0mm_P5.08mm_Vertical, F.Cu at (-45.6, -110.5)
- added R-SCFOLLWS-3: 9K 6W, Resistor_THT:R_Axial_DIN0516_L15.5mm_D5.0mm_P5.08mm_Vertical, F.Cu at (10.3, -166.9)
- added R-SCFOLLWS-4: 470, Resistor_THT:R_Axial_DIN0516_L15.5mm_D5.0mm_P5.08mm_Vertical, F.Cu at (-23.9, -138.6)
- added R-SCFOLLWS-5: 7K5 6W, Resistor_THT:R_Axial_DIN0516_L15.5mm_D5.0mm_P5.08mm_Vertical, F.Cu at (3.23, -152.4)
- added R-SCFOLLWS-6: 470, Resistor_THT:R_Axial_DIN0516_L15.5mm_D5.0mm_P5.08mm_Vertical, F.Cu at (-45.6, -104.0)
- added R-SCFOLLWS-7: 10K 6W, Resistor_THT:R_Axial_DIN0516_L15.5mm_D5.0mm_P5.08mm_Vertical, F.Cu at (-50.6, -88.6)
- added R-SCFOLLWS-8: 470K, Resistor_THT:R_Axial_DIN0516_L15.5mm_D5.0mm_P5.08mm_Vertical, F.Cu at (3.23, -145.8)
- added R-SCFOLLWS-9: 470, Resistor_THT:R_Axial_DIN0516_L15.5mm_D5.0mm_P5.08mm_Vertical, F.Cu at (-35.2, -110.5)
- added SW-DCHTRPU-1: SW_SPDT, Connector_PinHeader_2.54mm:PinHeader_1x03_P2.54mm_Vertical, F.Cu at (350.9, -9.44)
- added SW-KEYSW2-4: SW_Push_DPDT, Connector_PinHeader_2.54mm:PinHeader_1x06_P2.54mm_Vertical, F.Cu at (486.2, 55.2)
- added U-CMOSCRT1-9: 4049, Package_DIP:DIP-14_W7.62mm, F.Cu at (564.1, -197.1)
- added U-CMOSCRT2-7: 74LS00, Package_DIP:DIP-14_W7.62mm, F.Cu at (273.8, -61.4)
- added U-CRTPCIF2-2: SN75188N, localp:DIP794W53P254L1930H508Q14N, F.Cu at (-83.1, 186.1)
- added U-KVPSU1-1: VU111, NewValves:Valve_B4+1, F.Cu at (214.1, 186.1)
- added V-ADDER1-5: VR91, NewValves:Valve_9Loctal, F.Cu at (-284.4, -294.3)
- added V-CRTAMP4-3: CV173, NewValves:Valve_9Loctal, F.Cu at (-152.0, 46.0)
- added V-CRTCCT3-1: VCR97, NewValves:B12D, F.Cu at (186.8, 31.8)
- added V-CTRLGATE-4: VR91, NewValves:Valve_9Loctal, F.Cu at (-341.9, 184.6)
- added V-IGYSH3-4: VR91, NewValves:Valve_9Loctal, F.Cu at (-313.2, -0.91)
- added V-L-STAT-7: VR91, NewValves:Valve_9Loctal, F.Cu at (256.2, -236.8)
- added V-MONSW-6: VR91, NewValves:Valve_9Loctal, F.Cu at (-92.6, -265.6)
- added V-PREPULSE-3: VR91, NewValves:Valve_9Loctal, F.Cu at (-313.2, -140.2)
- added V-RMONDRS-6: EF50, NewValves:Valve_9Loctal, F.Cu at (-94.5, -58.5)
- added V-SCFOLLWS-1: CV173, NewValves:Valve_9Loctal, F.Cu at (-147.9, -140.2)
- added V-SCFOLLWS-10: CV173, NewValves:Valve_9Loctal, F.Cu at (-147.9, -168.9)
- added V-SCFOLLWS-2: CV173, NewValves:Valve_9Loctal, F.Cu at (-119.1, -168.9)
- added V-SCFOLLWS-3: CV173, NewValves:Valve_9Loctal, F.Cu at (-147.9, -111.4)
- added V-SCFOLLWS-4: CV173, NewValves:Valve_9Loctal, F.Cu at (-119.1, -140.2)
- added V-SCFOLLWS-5: CV173, NewValves:Valve_9Loctal, F.Cu at (-90.3, -168.9)
- added V-SCFOLLWS-6: CV173, NewValves:Valve_9Loctal, F.Cu at (-119.1, -111.4)
- added V-SCFOLLWS-7: CV173, NewValves:Valve_9Loctal, F.Cu at (-90.3, -140.2)
- added V-SCFOLLWS-8: CV173, NewValves:Valve_9Loctal, F.Cu at (-61.5, -168.9)
- added V-SCFOLLWS-9: CV173, NewValves:Valve_9Loctal, F.Cu at (-90.3, -111.4)
- C-ACTN_WF-3: renamed from R-FSTAT14-5; value 560K -> 100pf; footprint Resistor_THT:R_Axial_DIN0516_L15.5mm_D5.0mm_P5.08mm_Vertical -> Capacitor_THT:C_Disc_D7.5mm_W5.0mm_P5.00mm
- C-CMOSCRT1-4: renamed from R-IGYSH3-10; value 330K -> 100uf; footprint Resistor_THT:R_Axial_DIN0516_L15.5mm_D5.0mm_P5.08mm_Vertical -> Capacitor_THT:C_Disc_D7.5mm_W5.0mm_P5.00mm
- C-CRTAMP3-20: renamed from R-KVPSU2-3; value 800K -> 270pf; footprint Resistor_THT:R_Axial_DIN0516_L15.5mm_D5.0mm_P5.08mm_Vertical -> Capacitor_THT:C_Disc_D7.5mm_W5.0mm_P5.00mm
- C-CRTAMP3-35: renamed from R-L-STAT-18; value 180K -> 750p; footprint Resistor_THT:R_Axial_DIN0516_L15.5mm_D5.0mm_P5.08mm_Vertical -> Capacitor_THT:C_Disc_D7.5mm_W5.0mm_P5.00mm
- C-CRTAMP3-5: renamed from R-KVPSU1-6; value 2R 3W -> 10u; footprint Resistor_THT:R_Axial_DIN0516_L15.5mm_D5.0mm_P5.08mm_Vertical -> Capacitor_THT:C_Disc_D7.5mm_W5.0mm_P5.00mm
- C-CRTAMP4-17: renamed from R-MONSW-15; value 330K -> 0.1; footprint Resistor_THT:R_Axial_DIN0516_L15.5mm_D5.0mm_P5.08mm_Vertical -> Capacitor_THT:C_Disc_D7.5mm_W5.0mm_P5.00mm
- C-CRTAMP4-2: renamed from R-MONICCT-4; value 470K -> 0.5; footprint Resistor_THT:R_Axial_DIN0516_L15.5mm_D5.0mm_P5.08mm_Vertical -> Capacitor_THT:C_Disc_D7.5mm_W5.0mm_P5.00mm
- C-CRTAMP4-32: renamed from R-PREPULSE-11; value 470 -> 2U2; footprint Resistor_THT:R_Axial_DIN0516_L15.5mm_D5.0mm_P5.08mm_Vertical -> Capacitor_THT:C_Disc_D7.5mm_W5.0mm_P5.00mm
- C-CRTAMP4-47: renamed from R-PREPULSE-30; value 10K 3W -> 0.5; footprint Resistor_THT:R_Axial_DIN0516_L15.5mm_D5.0mm_P5.08mm_Vertical -> Capacitor_THT:C_Disc_D7.5mm_W5.0mm_P5.00mm
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Connections:
- C-ACTN_WF-3 pad 1: Net-(R-FSTAT14-1-Pad1) -> Net-(C-ACTN_WF-3-Pad1)
- C-ACTN_WF-3 pad 2: Net-(D-FSTAT14-3-Pad2) -> Net-(C-ACTN_WF-3-Pad2)
- C-CMOSCRT1-4 pad 1: Net-(C-IGYSH3-2-Pad1) -> Vdd
- C-CMOSCRT1-4 pad 2: /IGYSH3/-150V -> Vss
- C-CRTAMP3-20 pad 1: Net-(C-KVPSU2-2-Pad1) -> /CRTAMP3/GND
- C-CRTAMP3-20 pad 2: Net-(C-KVPSU2-2-Pad2) -> /CRTAMP3/Heater-6.3V
- C-CRTAMP3-35 pad 1: /L-STAT/GND -> Net-(C-CRTAMP3-1-Pad1)
- C-CRTAMP3-35 pad 2: Net-(C-L-STAT-7-Pad1) -> Net-(C-CRTAMP3-35-Pad2)
- C-CRTAMP3-5 pad 1: Net-(R-KVPSU1-6-Pad1) -> Net-(C-CRTAMP3-4-Pad2)
- C-CRTAMP3-5 pad 2: Net-(C-KVPSU1-4-Pad1) -> /CRTAMP3/GND
- C-CRTAMP4-17 pad 1: Net-(D-MONSW-2-Pad4) -> Net-(C-CRTAMP4-14-Pad2)
- C-CRTAMP4-17 pad 2: /MONSW/+200V -> /CRTAMP4/GND
- C-CRTAMP4-2 pad 1: Net-(C-MONICCT-1-Pad1) -> /CRTAMP4/+300
- C-CRTAMP4-2 pad 2: Net-(R-MONICCT-4-Pad2) -> /CRTAMP4/GND
- C-CRTAMP4-32 pad 1: Net-(R-PREPULSE-11-Pad1) -> Net-(C-CRTAMP4-32-Pad1)
- C-CRTAMP4-32 pad 2: Net-(R-PREPULSE-11-Pad2) -> /CRTAMP4/GND
- C-CRTAMP4-47 pad 1: Net-(R-PREPULSE-30-Pad1) -> /CRTAMP4/-150V
- C-CRTAMP4-47 pad 2: Net-(D-PREPULSE-18-Pad4) -> /CRTAMP4/GND
- C-CRTCCT4-5 pad 1: /PSEPCTL/+300V -> /CRTCCT4/Heater-6.3V
- C-CRTCCT4-5 pad 2: Net-(C-PSEPCTL-4-Pad1) -> /CRTCCT4/S.EHT(800-1400V)
- C-CRTPCIF2-6 pad 1: /RMONDRS/+300V -> Net-(C-CRTPCIF2-6-Pad1)
- C-CRTPCIF2-6 pad 2: Net-(D-RMONDRS-1-Pad2) -> Net-(C-CRTPCIF2-6-Pad2)
- C-CTRLGATE-9 pad 1: Net-(C-RMONDRS-11-Pad2) -> Net-(C-CTRLGATE-9-Pad1)
- C-CTRLGATE-9 pad 2: /RMONDRS/GND -> /CTRLGATE/GND
- C-FSTAT15-10 pad 1: /DCHTRPU/6V-DC -> /FSTAT15/-14V
- C-FSTAT15-10 pad 2: Net-(MES-DCHTRPU-1-Pad1) -> /FSTAT15/-150V
- C-IGYSH3-8 pad 1: (no net) -> Net-(C-IGYSH3-8-Pad1)
- C-IGYSH3-8 pad 2: (no net) -> Net-(C-IGYSH3-2-Pad2)
- C-PREPULSE-7 pad 1: (no net) -> Net-(C-PREPULSE-7-Pad1)
- C-PREPULSE-7 pad 2: (no net) -> Net-(C-PREPULSE-7-Pad2)
- C-PSEPCTL-6 pad 1: Net-(R-CMOSCRT2-50-Pad2) -> /PSEPCTL/+50V
- C-PSEPCTL-6 pad 2: /CMOSCRT2/OE -> /PSEPCTL/GND
- C-RMONDRS-5 pad 1: (no net) -> /RMONDRS/GND
- C-RMONDRS-5 pad 2: Net-(U-CRTPCIF2-2-Pad2) -> /RMONDRS/-150V
- C-SCFOLLWS-1 pad 1: (no net) -> Net-(C-SCFOLLWS-1-Pad1)
- C-SCFOLLWS-1 pad 2: (no net) -> Net-(C-SCFOLLWS-1-Pad2)
- D-ADDER1-15 pad 1: Net-(C-CRTCCT3-7-Pad2) -> /ADDER1/Heater-6.3V
- D-ADDER1-15 pad 2: /CRTCCT3/Heater-6.3V -> Net-(D-ADDER1-15-Pad2)
- D-ADDER1-15 pad 3: /CRTCCT3/Heater-6.3V -> /ADDER1/Heater-GND
- D-ADDER1-15 pad 4: /CRTCCT3/Heater-GND -> Net-(D-ADDER1-15-Pad4)
- D-ADDER1-16A1 pad 1: /CTRLGATE/Heater-GND -> /ADDER1/Heater-6.3V
- D-ADDER1-16A1 pad 2: Net-(C-CTRLGATE-9-Pad1) -> Net-(D-ADDER1-15-Pad2)
- D-ADDER1-16A1 pad 3: Net-(D-CTRLGATE-8-Pad2) -> /ADDER1/Heater-GND
- D-ADDER1-16A1 pad 4: Net-(R-CTRLGATE-17-Pad1) -> Net-(D-ADDER1-16A1-Pad4)
- D-ADDER1-8 pad 1: /CRTAMP4/Heater-GND -> /ADDER1/Heater-6.3V
- D-ADDER1-8 pad 2: Net-(C-CRTAMP4-26-Pad1) -> Net-(D-ADDER1-8-Pad2)
- D-ADDER1-8 pad 3: Net-(C-CRTAMP4-1-Pad1) -> /ADDER1/Heater-GND
- D-ADDER1-8 pad 4: Net-(C-CRTAMP4-26-Pad2) -> Net-(D-ADDER1-4-Pad4)
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