File: KiCAD/POWRCTL6b.sch (KiCad schematic (older format))
At the start: 110 parts

Commit message: Finish powrctl6b
Likely wrong bit of it I didn't understand other bits seem wrong inthe orginal.



Signed-off-by: John Bradley <flypie@rocketmail.com>
Parts:
- removed C-POWRCTL6b-? (x3): 0.5uf 3kv, Capacitor_THT:C_Disc_D7.5mm_W5.0mm_P5.00mm, symbol Device:C
- removed C-POWRCTL6b-? (x2): 1.5uf 3kV, Capacitor_THT:C_Disc_D7.5mm_W5.0mm_P5.00mm, symbol Device:C
- removed C-POWRCTL6b-? (x4): 0.5, Capacitor_THT:C_Disc_D7.5mm_W5.0mm_P5.00mm, symbol Device:C
- removed unit 1 of CR-POWRCTL6b-B2
- removed unit 2 of CR-POWRCTL6b-B2
- removed unit 3 of CR-POWRCTL6b-B2
- removed unit 1 of CR-POWRCTL6b-B3
- removed unit 4 of CR-POWRCTL6b-B3
- removed unit 3 of CR-POWRCTL6b-B3
- removed F-POWRCTL6b-? (x2): 4A, Fuse:Fuse_Littelfuse_395Series, symbol Device:Fuse
- removed J-POWRCTL6b-?: JA77847, Connector_PinHeader_2.54mm:PinHeader_1x08_P2.54mm_Vertical, symbol Connector_Generic:Conn_01x08
- removed J-POWRCTL6b-? (x2): +4V L, SamacSys_Parts_l:242431, symbol Connector:Conn_01x01_Female
- removed J-POWRCTL6b-? (x2): +4V N, SamacSys_Parts_l:242431, symbol Connector:Conn_01x01_Female
- removed J-POWRCTL6b-?: L, SamacSys_Parts_l:242431, symbol Connector:Conn_01x01_Female
- removed J-POWRCTL6b-?: N, SamacSys_Parts_l:242431, symbol Connector:Conn_01x01_Female
- removed J-POWRCTL6b-? (x4): 5, SamacSys_Parts_l:242431, symbol Connector:Conn_01x01_Female
- removed J-POWRCTL6b-?: 0V, SamacSys_Parts_l:242431, symbol Connector:Conn_01x01_Female
- removed J-POWRCTL6b-?: S.EHT -KV, SamacSys_Parts_l:242431, symbol Connector:Conn_01x01_Female
- removed L-POWRCTL6b-?: 100h 20 mA, Connector_PinHeader_2.54mm:PinHeader_1x02_P2.54mm_Vertical, symbol Device:L_Core_Iron
- removed M-POWRCTL6b-?: Voltmeter_DC, Connector_PinHeader_2.54mm:PinHeader_1x02_P2.54mm_Vertical, symbol Device:Voltmeter_DC
- removed R-POWRCTL6b-? (x2): 470, Resistor_THT:R_Axial_DIN0516_L15.5mm_D5.0mm_P5.08mm_Vertical, symbol Device:R
- removed R-POWRCTL6b-? (x4): 2R 3W, Resistor_THT:R_Axial_DIN0516_L15.5mm_D5.0mm_P5.08mm_Vertical, symbol Device:R
- removed R-POWRCTL6b-?: 0R8 4W, Resistor_THT:R_Axial_DIN0516_L15.5mm_D5.0mm_P5.08mm_Vertical, symbol Device:R
- removed R-POWRCTL6b-? (x2): 470K, Resistor_THT:R_Axial_DIN0516_L15.5mm_D5.0mm_P5.08mm_Vertical, symbol Device:R
- removed R-POWRCTL6b-?: 1.5K, Resistor_THT:R_Axial_DIN0516_L15.5mm_D5.0mm_P5.08mm_Vertical, symbol Device:R
- removed R-POWRCTL6b-? (x2): 22K, Resistor_THT:R_Axial_DIN0516_L15.5mm_D5.0mm_P5.08mm_Vertical, symbol Device:R
- removed R-POWRCTL6b-? (x4): 15k 3W, Resistor_THT:R_Axial_DIN0516_L15.5mm_D5.0mm_P5.08mm_Vertical, symbol Device:R
- removed R-POWRCTL6b-? (x2): 470k, Resistor_THT:R_Axial_DIN0516_L15.5mm_D5.0mm_P5.08mm_Vertical, symbol Device:R
- removed R-POWRCTL6b-?: 47k 2W, Resistor_THT:R_Axial_DIN0516_L15.5mm_D5.0mm_P5.08mm_Vertical, symbol Device:R
- removed R-POWRCTL6b-?: 4.5m, Resistor_THT:R_Axial_DIN0207_L6.3mm_D2.5mm_P2.54mm_Vertical, symbol Device:R
- removed R-POWRCTL6b-?: 4.7k, Resistor_THT:R_Axial_DIN0516_L15.5mm_D5.0mm_P5.08mm_Vertical, symbol Device:R
- removed R-POWRCTL6b-?: 360k, Resistor_THT:R_Axial_DIN0516_L15.5mm_D5.0mm_P5.08mm_Vertical, symbol Device:R
- removed RV-POWRCTL6b-?: 500K WW, Potentiometer_THT:Potentiometer_Piher_PT-10-V05_Vertical, symbol Device:R_POT
- removed SW-POWRCTL6b-?: SW_SPST, Connector_PinHeader_2.54mm:PinHeader_1x04_P2.54mm_Vertical, symbol Switch:SW_SPST
- removed TR-POWRCTL6b-?: VARIAC, Connector_PinHeader_2.54mm:PinHeader_1x10_P2.54mm_Vertical, symbol local:VARIAC
- removed TR-POWRCTL6b-?: Transformer_1P_1S, Connector_PinHeader_2.54mm:PinHeader_1x04_P2.54mm_Vertical, symbol Device:Transformer_1P_1S
- removed TR-POWRCTL6b-?: Transformer_1P_4S, Connector_PinHeader_2.54mm:PinHeader_1x10_P2.54mm_Vertical, symbol local:Transformer_1P_4S
- removed U-POWRCTL6b-?: CV71, Connector_PinHeader_2.54mm:PinHeader_1x02_P2.54mm_Vertical, symbol NEWValves:CV71
- removed U-POWRCTL6b-?: VU111, NewValves:Valve_B4+1, symbol NEWValves:VU111
- removed V-POWRCTL6b-?: CV73, NewValves:Valve_9Loctal, symbol NEWValves:CV73
- removed V-POWRCTL6b-? (x2): VR91, NewValves:Valve_9Loctal, symbol NEWValves:VR91
- added F-POWRCTL6b-1: 1A, Connector_PinHeader_2.54mm:PinHeader_1x02_P2.54mm_Vertical, symbol Device:Fuse
- added F-POWRCTL6b-2: 4A, Connector_PinHeader_2.54mm:PinHeader_1x02_P2.54mm_Vertical, symbol Device:Fuse
- added F-POWRCTL6b-5: Fuse, Connector_PinHeader_2.54mm:PinHeader_1x02_P2.54mm_Vertical, symbol Device:Fuse
- added J-POWRCTL6b-10, J-POWRCTL6b-11, J-POWRCTL6b-35, J-POWRCTL6b-37, J-POWRCTL6b-40, J-POWRCTL6b-42: 3, TerminalBlock_MetzConnect:TerminalBlock_MetzConnect_360271_1x01_Horizontal_ScrewM3.0_Boxed, symbol Connector:Screw_Terminal_01x01
- added J-POWRCTL6b-13, J-POWRCTL6b-18, J-POWRCTL6b-33, J-POWRCTL6b-38: 5, TerminalBlock_MetzConnect:TerminalBlock_MetzConnect_360271_1x01_Horizontal_ScrewM3.0_Boxed, symbol Connector:Screw_Terminal_01x01
- added J-POWRCTL6b-14, J-POWRCTL6b-34, J-POWRCTL6b-39: 4, TerminalBlock_MetzConnect:TerminalBlock_MetzConnect_360271_1x01_Horizontal_ScrewM3.0_Boxed, symbol Connector:Screw_Terminal_01x01
- added J-POWRCTL6b-15: 6, TerminalBlock_MetzConnect:TerminalBlock_MetzConnect_360271_1x01_Horizontal_ScrewM3.0_Boxed, symbol Connector:Screw_Terminal_01x01
- added J-POWRCTL6b-16, J-POWRCTL6b-19: 7, TerminalBlock_MetzConnect:TerminalBlock_MetzConnect_360271_1x01_Horizontal_ScrewM3.0_Boxed, symbol Connector:Screw_Terminal_01x01
- added J-POWRCTL6b-17, J-POWRCTL6b-22: 10, TerminalBlock_MetzConnect:TerminalBlock_MetzConnect_360271_1x01_Horizontal_ScrewM3.0_Boxed, symbol Connector:Screw_Terminal_01x01
- added J-POWRCTL6b-20, J-POWRCTL6b-21: 8, TerminalBlock_MetzConnect:TerminalBlock_MetzConnect_360271_1x01_Horizontal_ScrewM3.0_Boxed, symbol Connector:Screw_Terminal_01x01
- added J-POWRCTL6b-23, J-POWRCTL6b-24, J-POWRCTL6b-27, J-POWRCTL6b-28, J-POWRCTL6b-29, J-POWRCTL6b-30, J-POWRCTL6b-31, J-POWRCTL6b-32: (no value), TerminalBlock_MetzConnect:TerminalBlock_MetzConnect_360271_1x01_Horizontal_ScrewM3.0_Boxed, symbol Connector:Screw_Terminal_01x01
- added J-POWRCTL6b-25: 12, TerminalBlock_MetzConnect:TerminalBlock_MetzConnect_360271_1x01_Horizontal_ScrewM3.0_Boxed, symbol Connector:Screw_Terminal_01x01
- added J-POWRCTL6b-26: 11, TerminalBlock_MetzConnect:TerminalBlock_MetzConnect_360271_1x01_Horizontal_ScrewM3.0_Boxed, symbol Connector:Screw_Terminal_01x01
- added J-POWRCTL6b-36, J-POWRCTL6b-41, J-POWRCTL6b-8, J-POWRCTL6b-9: 2, TerminalBlock_MetzConnect:TerminalBlock_MetzConnect_360271_1x01_Horizontal_ScrewM3.0_Boxed, symbol Connector:Screw_Terminal_01x01
- added J-POWRCTL6b-6, J-POWRCTL6b-7: 1, TerminalBlock_MetzConnect:TerminalBlock_MetzConnect_360271_1x01_Horizontal_ScrewM3.0_Boxed, symbol Connector:Screw_Terminal_01x01
- added MES-POWRCTL6b-1, MES-POWRCTL6b-5, MES-POWRCTL6b-6, MES-POWRCTL6b-7: 7V, Connector_PinHeader_2.54mm:PinHeader_1x02_P2.54mm_Vertical, symbol Device:Voltmeter_AC
- added MES-POWRCTL6b-4: 5A, Connector_PinHeader_2.54mm:PinHeader_1x02_P2.54mm_Vertical, symbol Device:Amperemeter_AC
- added R-POWRCTL6b-3: 2R 3W, Resistor_THT:R_Axial_DIN0516_L15.5mm_D5.0mm_P5.08mm_Vertical, symbol Device:R
- added RV-POWRCTL6b-3: 17R, Connector_PinHeader_2.54mm:PinHeader_1x03_P2.54mm_Vertical, symbol Device:R_POT_TRIM
- added SW-POWRCTL6b-1: SW_SPST, Connector_PinHeader_2.54mm:PinHeader_1x04_P2.54mm_Vertical, symbol Switch:SW_SPST
- added SW-POWRCTL6b-2: SW_Push, Connector_PinHeader_2.54mm:PinHeader_1x02_P2.54mm_Vertical, symbol Switch:SW_Push
- added SW-POWRCTL6b-3: SW_Push_Open, Connector_PinHeader_2.54mm:PinHeader_1x02_P2.54mm_Vertical, symbol Switch:SW_Push_Open
- added SW-POWRCTL6b-6: SW_SPDT, Connector_PinHeader_2.54mm:PinHeader_1x03_P2.54mm_Vertical, symbol Switch:SW_SPDT
- added T-POWRCTL6b-1, T-POWRCTL6b-2: Transformer_1P_2S, Connector_PinHeader_2.54mm:PinHeader_1x06_P2.54mm_Vertical, symbol Device:Transformer_1P_2S
- added V-POWRCTL6b-4: CV71, Connector_PinHeader_2.54mm:PinHeader_1x02_P2.54mm_Vertical, symbol NEWValves:CV71
- CB-POWRCTL6b-1: renamed from CB-POWRCTL6b-?; footprint (none) -> Connector_PinHeader_2.54mm:PinHeader_1x06_P2.54mm_Vertical
- CR-POWRCTL6b-1, CR-POWRCTL6b-4, CR-POWRCTL6b-A3: footprint (none) -> Connector_PinHeader_2.54mm:PinHeader_1x10_P2.54mm_Vertical
- CR-POWRCTL6b-1, CR-POWRCTL6b-4: footprint (none) -> Connector_PinHeader_2.54mm:PinHeader_1x10_P2.54mm_Vertical; symbol NEWValves:DILA-22(230V50HZ,240V60HZ) -> ContactorRelay:DILA-22
- CR-POWRCTL6b-A2: value DILA-22 -> DILA-40; footprint (none) -> Connector_PinHeader_2.54mm:PinHeader_1x10_P2.54mm_Vertical
- CR-POWRCTL6b-A2: value DILA-22 -> DILA-40; footprint (none) -> Connector_PinHeader_2.54mm:PinHeader_1x10_P2.54mm_Vertical; symbol NEWValves:DILA-22(230V50HZ,240V60HZ) -> ContactorRelay:DILA-40
- CR-POWRCTL6b-B2: value DILA-XHI22 -> DILA-XHI10; footprint (none) -> Connector_PinHeader_2.54mm:PinHeader_1x10_P2.54mm_Vertical; symbol ContactorRelay:DILA-XHI22 -> ContactorRelay:DILA-XHI10
- CR-POWRCTL6b-B3: value DILA-XHI22 -> DILA-XHI01; footprint (none) -> Connector_PinHeader_2.54mm:PinHeader_1x10_P2.54mm_Vertical; symbol ContactorRelay:DILA-XHI22 -> ContactorRelay:DILA-XHI01
- D-POWRCTL6b-1, D-POWRCTL6b-10, D-POWRCTL6b-11, D-POWRCTL6b-12, D-POWRCTL6b-13, D-POWRCTL6b-14, D-POWRCTL6b-15, D-POWRCTL6b-16, D-POWRCTL6b-17, D-POWRCTL6b-18, D-POWRCTL6b-2, D-POWRCTL6b-3, D-POWRCTL6b-4, D-POWRCTL6b-5, D-POWRCTL6b-6, D-POWRCTL6b-7, D-POWRCTL6b-8, D-POWRCTL6b-9: renamed from D-POWRCTL6b-?; footprint (none) -> Package_TO_SOT_THT:TO-46-2
- F-POWRCTL6b-3, F-POWRCTL6b-4: renamed from F-POWRCTL6b-?; footprint (none) -> Connector_PinHeader_2.54mm:PinHeader_1x02_P2.54mm_Vertical
- J-POWRCTL6b-1, J-POWRCTL6b-2, J-POWRCTL6b-3, J-POWRCTL6b-4, J-POWRCTL6b-5: renamed from J-POWRCTL6b-?; footprint (none) -> TerminalBlock_MetzConnect:TerminalBlock_MetzConnect_360271_1x01_Horizontal_ScrewM3.0_Boxed
- J-POWRCTL6b-12: renamed from J-POWRCTL6b-?; footprint (none) -> Connector_PinHeader_2.54mm:PinHeader_1x02_P2.54mm_Vertical
- MES-POWRCTL6b-2, MES-POWRCTL6b-3: renamed from MES-POWRCTL6b-?; footprint (none) -> Connector_PinHeader_2.54mm:PinHeader_1x02_P2.54mm_Vertical
- P-POWRCTL6b-1: renamed from P-POWRCTL6b-?; footprint (none) -> Connector_PinHeader_2.54mm:PinHeader_1x02_P2.54mm_Vertical
- PSU-POWRCTL6b-1, PSU-POWRCTL6b-2, PSU-POWRCTL6b-3, PSU-POWRCTL6b-4, PSU-POWRCTL6b-5, PSU-POWRCTL6b-6: renamed from PSU-POWRCTL6b-?; footprint (none) -> Connector_PinHeader_2.54mm:PinHeader_1x09_P2.54mm_Vertical
- RV-POWRCTL6b-1, RV-POWRCTL6b-2: renamed from RV-POWRCTL6b-?; footprint (none) -> Connector_PinHeader_2.54mm:PinHeader_1x03_P2.54mm_Vertical
- SW-POWRCTL6b-4, SW-POWRCTL6b-5: renamed from SW-POWRCTL6b-?; footprint (none) -> Connector_PinHeader_2.54mm:PinHeader_1x03_P2.54mm_Vertical
- TR-POWRCTL6b-1: renamed from TR-POWRCTL6b-?; footprint (none) -> Connector_PinHeader_2.54mm:PinHeader_1x03_P2.54mm_Vertical
- V-POWRCTL6b-1, V-POWRCTL6b-2, V-POWRCTL6b-3: renamed from U-POWRCTL6b-?; footprint (none) -> Connector_PinHeader_2.54mm:PinHeader_1x02_P2.54mm_Vertical
- gave numbers to parts that had none: 2
Connections:
- net labels added: +50, -150, 0V, 0Vbar
- net labels removed: -150*, 200*, 6.3V-L, 6.3V-N
- wire segments 383 -> 378
- no-connect marks 4 -> 9
Other:
- note added: "-150 Margins"
- note added: "6.5V 50A"
- note added: "HT Rack"
- note added: "Heater Transformers Panel"
- note added: "Meters Panel"
- note added: "NOTE: The heaters load on the two transformers should be reasonably\nwell balanced: as between the halves of the windings because\nthe centre tap is not able to carry more than about 20A, and\nbetween the two transformers so that on standby (heaters OFF),\nall heaters run at about half voltage."
- note added: "Power Inlet Panel"
- note added: "Supp. OK link\noriginally connected\nbetween 5 & 6"
- note removed: "2KV"
- note removed: "4.1v 1A"
- note removed: "4v 3A\nfor CV73"
- note removed: "6.3v 2A"
- note removed: "Aux Supply"
- note removed: "NOTE.\nTwo supplies are needed - one for the storage tubes, the other for the monitor tube.\nTwo diferent units are shown on photo AAR10, with differeing meter arrangements.\nThe above circuit may be adapted for the two different uses.\nThe regulator valve must have enough, but not excessive, voltage across it.\nThe neon should be alight (>300V), but not excessively bright (>700V).\nSee separate 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"
- note removed: "Variac"
- moved on the sheet: CR-POWRCTL6b-1A, CR-POWRCTL6b-1B, CR-POWRCTL6b-1C, CR-POWRCTL6b-1D, CR-POWRCTL6b-1E, CR-POWRCTL6b-4A, CR-POWRCTL6b-4E, CR-POWRCTL6b-A2A, CR-POWRCTL6b-A2D, CR-POWRCTL6b-A2E, CR-POWRCTL6b-A3E, F-POWRCTL6b-3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
