File: KiCAD/STAB200.sch (KiCad schematic (older format))
At the start: 31 parts

Commit message: Add StorGate & some Valve Logic data.
Signed-off-by: John Bradley <flypie@rocketmail.com>
Parts:
- removed C-SMONXTB-5, C-SMONXTB-7: 0.5, Capacitor_THT:C_Disc_D7.5mm_W5.0mm_P5.00mm, symbol Device:C
- removed unit 2 of V-SMONXTB-2
- added C-STAB200-5, C-STAB200-7: 0.5, Capacitor_THT:C_Disc_D7.5mm_W5.0mm_P5.00mm, symbol Device:C
- added unit 2 of V-STAB200-2
- V-STAB200-1: renamed from V-SMONXTB-1; symbol NEWValves:VR91 -> NEWValves:807
- renumbered C-SMONXTB-1 to C-STAB200-1, C-SMONXTB-2 to C-STAB200-2, C-SMONXTB-3 to C-STAB200-3, C-SMONXTB-4 to C-STAB200-4, C-SMONXTB-8 to C-STAB200-8, D-SMONXTB-3 to D-STAB200-3, MES-SMONXTB-1 to MES-STAB200-1, MES-SMONXTB-2 to MES-STAB200-2, P-SMONXTB-1 to P-STAB200-1, R-SMONXTB-1 to R-STAB200-1, R-SMONXTB-10 to R-STAB200-10, R-SMONXTB-11 to R-STAB200-11, R-SMONXTB-12 to R-STAB200-12, R-SMONXTB-13 to R-STAB200-13, R-SMONXTB-14 to R-STAB200-14, R-SMONXTB-2 to R-STAB200-2, R-SMONXTB-3 to R-STAB200-3, R-SMONXTB-4 to R-STAB200-4, R-SMONXTB-5 to R-STAB200-5, R-SMONXTB-6 to R-STAB200-6, R-SMONXTB-7 to R-STAB200-7, R-SMONXTB-8 to R-STAB200-8, R-SMONXTB-9 to R-STAB200-9, RV-SMONXTB-1 to RV-STAB200-1, T-SMONXTB-1 to T-STAB200-1, V-SMONXTB-1 to V-STAB200-1, V-SMONXTB-2 to V-STAB200-2, V-SMONXTB-3 to V-STAB200-3
Connections:
- net +0V: now also C-STAB200-5.2, C-STAB200-7.1
- net +200V: now also C-STAB200-5.1
- net -150V: now also C-STAB200-7.2
- net Heater-6.3V: now also V-STAB200-1.5 (F1), V-STAB200-2.9 (H); no longer V-STAB200-1.9 (H)
- net Heater-GND: now also V-STAB200-2.1 (H)
