File: KiCAD/STORGATE.sch (KiCad schematic (older format))
At the start: 71 parts

Commit message: Add SUBTR1.sch, SXTMBASE.sch TRANSFER.sch.
Signed-off-by: John Bradley <flypie@rocketmail.com>
Parts:
- added J-STORGATE-2: HIGH Voltage., Connector_TE-Connectivity:TE_MATE-N-LOK_1-770972-x_2x06_P4.14mm_Horizontal, symbol Connector_Generic:Conn_02x06_Odd_Even
- gave numbers to parts that had none: 1
Connections:
- net +200V: now also J-STORGATE-2.2 (Pin_2)
- net +300V: now also J-STORGATE-2.1 (Pin_1)
- net +50V: now also J-STORGATE-2.3 (Pin_3)
- net -150V: now also J-STORGATE-2.4 (Pin_4)
- net GND: now also J-STORGATE-2.5 (Pin_5), J-STORGATE-2.6 (Pin_6)
- net Heater-6.3V: now also J-STORGATE-2.12 (Pin_12)
- net Heater-GND: now also J-STORGATE-2.11 (Pin_11)
- no-connect marks 10 -> 14
Changed lines of the file:
@@
 $Descr A3 16535 11693
 encoding utf-8
-Sheet 39 39
+Sheet 39 42
 Title "Store Gate Position 6.6"
 Date "2020-10-15"
@@
 $Comp
 L NEWValves:VR91 V-STORGATE-1
-U 2 1 5FFCCC3B
+U 2 1 5F8CD19C
 P 1300 10450
 F 0 "V-STORGATE-1" H 1300 11025 50  0000 C CNN
@@
 $Comp
 L Device:C C-STORGATE-4
-U 1 1 5FFCCC34
+U 1 1 5F8CD19B
 P 8750 10550
 F 0 "C-STORGATE-4" H 8900 10625 50  0000 L CNN
@@
 $Comp
 L NEWValves:VR91 V-STORGATE-3
-U 2 1 5FE20AD4
+U 2 1 5F8CD18D
 P 2600 10450
 F 0 "V-STORGATE-3" H 2600 11025 50  0000 C CNN
@@
 $Comp
 L NEWValves:EA50 D-SCFOLLWS-?
-U 2 1 5F9334CE
+U 2 1 5F8CD18A
 P 1300 9050
-AR Path="/5F868E46/5F9334CE" Ref="D-SCFOLLWS-?"  Part="1"
-AR Path="/5F89590E/5F9334CE" Ref="D-STORGATE-1"  Part="2"
-AR Path="/5FFFB333/5F9334CE" Ref="D-STORGATE-1"  Part="2"
+AR Path="/5F868E46/5F8CD18A" Ref="D-SCFOLLWS-?"  Part="1"
+AR Path="/5F89590E/5F8CD18A" Ref="D-STORGATE-1"  Part="2"
+AR Path="/5FFFB333/5F8CD18A" Ref="D-STORGATE-1"  Part="2"
 F 0 "D-STORGATE-1" H 1300 9350 50  0000 C CNN
 F 1 "EA50" H 1300 9250 50  0000 C CNN
@@
 	11000 10800 11000 10700
 $Comp
-L Switch:SW_SPDT SW-STORGATE-?
+L Switch:SW_SPDT SW-STORGATE-1
 U 1 1 600456EE
 P 1800 4000
-F 0 "SW-STORGATE-?" H 1800 4300 50  0000 C CNN
+F 0 "SW-STORGATE-1" H 1800 4300 50  0000 C CNN
 F 1 "SW_SPDT" H 1800 4200 50  0000 C CNN
 F 2 "Connector_PinSocket_2.54mm:PinSocket_1x03_P2.54mm_Vertical" H 1800 4000 50  0001 C CNN
@@
 $Comp
 L Connector:Conn_01x01_Female J-STORGATE-?
-U 1 1 6007891E
+U 1 1 5F8CD19D
 P 1250 4550
-AR Path="/5F88E8BA/6007891E" Ref="J-STORGATE-?"  Part="1"
-AR Path="/5F89590E/6007891E" Ref="J-STORGATE-?"  Part="1"
-AR Path="/5FFFB333/6007891E" Ref="J-STORGATE-11"  Part="1"
+AR Path="/5F88E8BA/5F8CD19D" Ref="J-STORGATE-?"  Part="1"
+AR Path="/5F89590E/5F8CD19D" Ref="J-STORGATE-?"  Part="1"
+AR Path="/5FFFB333/5F8CD19D" Ref="J-STORGATE-11"  Part="1"
 F 0 "J-STORGATE-11" H 1300 4450 50  0000 L CNN
 F 1 "S.Dummy.Sig" H 1300 4550 50  0000 L CNN
@@
 $Comp
 L NEWValves:CV173 V-STORGATE-5
-U 2 1 5FDBE41C
+U 2 1 5F8CD18B
 P 3900 10450
 F 0 "V-STORGATE-5" H 3900 11025 50  0000 C CNN
@@
 $Comp
 L NEWValves:VR91 V-STORGATE-6
-U 2 1 5FDBE8C2
+U 2 1 5F8CD18C
 P 4550 10450
 F 0 "V-STORGATE-6" H 4550 11025 50  0000 C CNN
@@
 $Comp
 L NEWValves:EA50 D-STORGATE-?
-U 2 1 5FE6039A
+U 2 1 5F8CD194
 P 5200 9050
-AR Path="/5F868E46/5FE6039A" Ref="D-STORGATE-?"  Part="1"
-AR Path="/5F89590E/5FE6039A" Ref="D-STORGATE-?"  Part="2"
-AR Path="/5FFFB333/5FE6039A" Ref="D-STORGATE-8"  Part="2"
+AR Path="/5F868E46/5F8CD194" Ref="D-STORGATE-?"  Part="1"
+AR Path="/5F89590E/5F8CD194" Ref="D-STORGATE-?"  Part="2"
+AR Path="/5FFFB333/5F8CD194" Ref="D-STORGATE-8"  Part="2"
 F 0 "D-STORGATE-8" H 5200 9350 50  0000 C CNN
 F 1 "EA50" H 5200 9250 50  0000 C CNN
@@
 $Comp
 L NEWValves:EA50 D-STORGATE-?
-U 2 1 5FE603AA
+U 2 1 5F8CD195
 P 4550 9050
-AR Path="/5F868E46/5FE603AA" Ref="D-STORGATE-?"  Part="1"
-AR Path="/5F89590E/5FE603AA" Ref="D-STORGATE-?"  Part="2"
-AR Path="/5FFFB333/5FE603AA" Ref="D-STORGATE-7"  Part="2"
+AR Path="/5F868E46/5F8CD195" Ref="D-STORGATE-?"  Part="1"
+AR Path="/5F89590E/5F8CD195" Ref="D-STORGATE-?"  Part="2"
+AR Path="/5FFFB333/5F8CD195" Ref="D-STORGATE-7"  Part="2"
 F 0 "D-STORGATE-7" H 4550 9350 50  0000 C CNN
 F 1 "EA50" H 4550 9250 50  0000 C CNN
@@
 $Comp
 L NEWValves:EA50 D-STORGATE-?
-U 2 1 5FE8663C
+U 2 1 5F8CD199
 P 7800 9050
-AR Path="/5F868E46/5FE8663C" Ref="D-STORGATE-?"  Part="1"
-AR Path="/5F89590E/5FE8663C" Ref="D-STORGATE-?"  Part="2"
-AR Path="/5FFFB333/5FE8663C" Ref="D-STORGATE-16"  Part="2"
+AR Path="/5F868E46/5F8CD199" Ref="D-STORGATE-?"  Part="1"
+AR Path="/5F89590E/5F8CD199" Ref="D-STORGATE-?"  Part="2"
+AR Path="/5FFFB333/5F8CD199" Ref="D-STORGATE-16"  Part="2"
 F 0 "D-STORGATE-16" H 7800 9350 50  0000 C CNN
 F 1 "EA50" H 7800 9250 50  0000 C CNN
@@
 $Comp
 L NEWValves:EA50 D-STORGATE-?
-U 2 1 5FE8664A
+U 2 1 5F8CD19A
 P 7150 9050
-AR Path="/5F868E46/5FE8664A" Ref="D-STORGATE-?"  Part="1"
-AR Path="/5F89590E/5FE8664A" Ref="D-STORGATE-?"  Part="2"
-AR Path="/5FFFB333/5FE8664A" Ref="D-STORGATE-15"  Part="2"
+AR Path="/5F868E46/5F8CD19A" Ref="D-STORGATE-?"  Part="1"
+AR Path="/5F89590E/5F8CD19A" Ref="D-STORGATE-?"  Part="2"
+AR Path="/5FFFB333/5F8CD19A" Ref="D-STORGATE-15"  Part="2"
 F 0 "D-STORGATE-15" H 7150 9350 50  0000 C CNN
 F 1 "EA50" H 7150 9250 50  0000 C CNN
@@
 Wire Wire Line
 	6700 6950 6700 7650
+$Comp
+L power:PWR_FLAG #FLG?
+U 1 1 5FCDF780
+P 12450 6350
+AR Path="/5F868E46/5FCDF780" Ref="#FLG?"  Part="1"
+AR Path="/5F2DDAEA/5FCDF780" Ref="#FLG?"  Part="1"
+AR Path="/60BC2C2A/5FCDF780" Ref="#FLG?"  Part="1"
+AR Path="/5F89117E/5FCDF780" Ref="#FLG?"  Part="1"
+AR Path="/5F88E8BA/5FCDF780" Ref="#FLG?"  Part="1"
+AR Path="/6077FCA5/5FCDF780" Ref="#FLG?"  Part="1"
+AR Path="/5F89590E/5FCDF780" Ref="#FLG?"  Part="1"
+AR Path="/5FFFB333/5FCDF780" Ref="#FLG0178"  Part="1"
+F 0 "#FLG0178" H 12450 6425 50  0001 C CNN
+F 1 "PWR_FLAG" H 12475 6550 50  0000 C CNN
+F 2 "" H 12450 6350 50  0001 C CNN
+F 3 "~" H 12450 6350 50  0001 C CNN
+	1    12450 6350
+	-1   0    0    1
+$EndComp
+Text Label 12500 5900 0    50   ~ 0
+-150V
+Wire Wire Line
+	12400 6300 12450 6300
+Text Label 12500 6300 0    50   ~ 0
+Heater-6.3V
+Connection ~ 12450 6300
+Wire Wire Line
+	12450 6300 12500 6300
+Wire Wire Line
+	12450 6350 12450 6300
+Text Label 12500 5800 0    50   ~ 0
++200V
+NoConn ~ 12400 6100
+NoConn ~ 12400 6200
+Wire Wire Line
+	12500 5800 12400 5800
+Text Label 12500 6000 0    50   ~ 0
+GND
+Wire Wire Line
+	12500 6000 12400 6000
+Wire Wire Line
+	12500 5900 12400 5900
+NoConn ~ 11900 6100
+NoConn ~ 11900 6200
+Text Label 11800 6300 2    50   ~ 0
+Heater-GND
+Wire Wire Line
+	11900 6000 11800 6000
+Wire Wire Line
+	11900 5900 11800 5900
+Wire Wire Line
+	11900 5800 11800 5800
+Wire Wire Line
+	11850 6300 11800 6300
+Connection ~ 11850 6300
+Wire Wire Line
+	11850 6350 11850 6300
+Wire Wire Line
+	11900 6300 11850 6300
+$Comp
+L power:PWR_FLAG #FLG?
+U 1 1 5FCDF79D
+P 11850 6350
+AR Path="/5F868E46/5FCDF79D" Ref="#FLG?"  Part="1"
+AR Path="/5F2DDAEA/5FCDF79D" Ref="#FLG?"  Part="1"
+AR Path="/60BC2C2A/5FCDF79D" Ref="#FLG?"  Part="1"
+AR Path="/5F89117E/5FCDF79D" Ref="#FLG?"  Part="1"
+AR Path="/5F88E8BA/5FCDF79D" Ref="#FLG?"  Part="1"
+AR Path="/6077FCA5/5FCDF79D" Ref="#FLG?"  Part="1"
+AR Path="/5F89590E/5FCDF79D" Ref="#FLG?"  Part="1"
+AR Path="/5FFFB333/5FCDF79D" Ref="#FLG0179"  Part="1"
+F 0 "#FLG0179" H 11850 6425 50  0001 C CNN
+F 1 "PWR_FLAG" H 11875 6550 50  0000 C CNN
+F 2 "" H 11850 6350 50  0001 C CNN
+F 3 "~" H 11850 6350 50  0001 C CNN
+	1    11850 6350
+	-1   0    0    1
+$EndComp
+Text Label 11800 6000 2    50   ~ 0
+GND
+Text Label 11800 5900 2    50   ~ 0
++50V
+Text Label 11800 5800 2    50   ~ 0
++300V
+$Comp
+L Connector_Generic:Conn_02x06_Odd_Even J-STOP-?
+U 1 1 5FCDF7A6
+P 12100 6000
+AR Path="/5F868E46/5FCDF7A6" Ref="J-STOP-?"  Part="1"
+AR Path="/5F2DDAEA/5FCDF7A6" Ref="J-STOP-?"  Part="1"
+AR Path="/60BC2C2A/5FCDF7A6" Ref="J-STOP-?"  Part="1"
+AR Path="/5F89117E/5FCDF7A6" Ref="J-STOP-?"  Part="1"
+AR Path="/5F88E8BA/5FCDF7A6" Ref="J-STOP-?"  Part="1"
+AR Path="/6077FCA5/5FCDF7A6" Ref="J-STOP-?"  Part="1"
+AR Path="/5F89590E/5FCDF7A6" Ref="J-STOP-?"  Part="1"
+AR Path="/5FFFB333/5FCDF7A6" Ref="J-STORGATE-2"  Part="1"
+F 0 "J-STORGATE-2" H 12150 6450 50  0000 C CNN
+F 1 "HIGH Voltage." H 12150 6350 50  0000 C CNN
+F 2 "Connector_TE-Connectivity:TE_MATE-N-LOK_1-770972-x_2x06_P4.14mm_Horizontal" H 12100 6000 50  0001 C CNN
+F 3 "~" H 12100 6000 50  0001 C CNN
+	1    12100 6000
+	1    0    0    -1
+$EndComp
 $EndSCHEMATC
