File: KiCAD/YAMP&HVR.sch (KiCad schematic (older format))
At the start: 67 parts

Commit message: Signed-off-by: John Bradley <flypie@rocketmail.com>
Parts:
- added G?: GNDFRM, symbol NEWValves:GNDFRM
Changed lines of the file:
@@
 U 1 1 62C9C2DB
 P 8150 1600
-F 0 "R-YAMP&HVR-31" V 8400 1600 50  0000 C CNN
-F 1 "47" V 8300 1600 50  0000 C CNN
+F 0 "R-YAMP&HVR-31" V 7950 1600 50  0000 C CNN
+F 1 "47" V 8050 1600 50  0000 C CNN
 F 2 "Resistor_THT:R_Axial_DIN0516_L15.5mm_D5.0mm_P5.08mm_Vertical" V 8080 1600 50  0001 C CNN
 F 3 "~" H 8150 1600 50  0001 C CNN
@@
 Wire Wire Line
 	9100 4650 9100 4750
-Text Label 9100 4750 0    50   ~ 0
-GND
 Wire Wire Line
 	9100 4250 8150 4250
@@
 	1    0    0    -1
 $EndComp
+$Comp
+L NEWValves:GNDFRM G?
+U 1 1 5F92EAEA
+P 9100 4750
+F 0 "G?" H 8950 4750 50  0001 C CNN
+F 1 "GNDFRM" H 9200 4750 50  0000 L CNN
+F 2 "" V 9100 4750 50  0001 C CNN
+F 3 "" V 9100 4750 50  0001 C CNN
+	1    9100 4750
+	1    0    0    -1
+$EndComp
